File: GE-Regs.kicad_sch (KiCad schematic)
At the start: 16 parts, among them J40 Vin, J41 Gnd, U50 SPX3819M5-L-3-3, U60 SY8113BADC

Commit message: all nets routed for next revision, no major drc errors
Parts:
- removed TP60: TestPoint, AlfredoFootprints:GE_TestPoint_Loop, symbol Connector:TestPoint
- R60: LCSC (none) -> C25741
- R61: LCSC (none) -> C25754
Changed lines of the file:
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@@
   (junction (at 210.82 115.57) (diameter 0) (color 0 0 0 0)
   )
-  (junction (at 218.44 107.95) (diameter 0) (color 0 0 0 0)
-  )
   (wire (pts (xy 95.25 91.44) (xy 100.33 91.44))
     (stroke (width 0) (type default) (color 0 0 0 0))
@@
     (stroke (width 0) (type default) (color 0 0 0 0))
   )
-  (wire (pts (xy 210.82 107.95) (xy 218.44 107.95))
+  (wire (pts (xy 210.82 107.95) (xy 226.06 107.95))
     (stroke (width 0) (type default) (color 0 0 0 0))
   )
@@
   )
   (wire (pts (xy 193.04 69.85) (xy 199.39 69.85))
-    (stroke (width 0) (type default) (color 0 0 0 0))
-  )
-  (wire (pts (xy 218.44 107.95) (xy 226.06 107.95))
     (stroke (width 0) (type default) (color 0 0 0 0))
   )
@@
       (effects (font (size 1.27 1.27)) hide)
     )
-    (property "LCSC" "" (id 4) (at 210.82 111.76 0)
+    (property "LCSC" "C25741" (id 4) (at 210.82 111.76 0)
       (effects (font (size 1.27 1.27)) hide)
     )
@@
       (effects (font (size 1.27 1.27)) hide)
     )
-    (property "LCSC" "" (id 4) (at 210.82 119.38 0)
+    (property "LCSC" "C25754" (id 4) (at 210.82 119.38 0)
       (effects (font (size 1.27 1.27)) hide)
     )
@@
       (effects (font (size 1.27 1.27)) hide)
     )
-    (pin "1")
-  )
-  (symbol (lib_id "Connector:TestPoint") (at 218.44 107.95 0) (unit 1)
-    (in_bom yes) (on_board yes)
-    (property "Reference" "TP60" (id 0) (at 214.63 102.87 0)
-      (effects (font (size 1.27 1.27)) (justify left))
-    )
-    (property "Value" "TestPoint" (id 1) (at 213.36 100.33 0)
-      (effects (font (size 1.27 1.27)) (justify left))
-    )
-    (property "Footprint" "AlfredoFootprints:GE_TestPoint_Loop" (id 2) (at 223.52 107.95 0)
-      (effects (font (size 1.27 1.27)) hide)
-    )
-    (property "Datasheet" "~" (id 3) (at 223.52 107.95 0)
-      (effects (font (size 1.27 1.27)) hide)
-    )
-    (property "LCSC" "~" (id 4) (at 218.44 107.95 0)
-      (effects (font (size 1.27 1.27)) hide)
-    )

Commit message: updated gitignore
Parts:
- C63: value 22uF, 10V -> 2.2uF, 10V
Changed lines of the file:
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@@
       (effects (font (size 1.27 1.27)) (justify right))
     )
-    (property "Value" "22uF, 10V" (id 1) (at 236.22 114.3 0)
+    (property "Value" "2.2uF, 10V" (id 1) (at 236.22 114.3 0)
       (effects (font (size 1.27 1.27)) (justify right))
     )
