File: I3ESC.kicad_sch (KiCad schematic)
At the start: 42 parts, among them J30 CanOut, J4 GND, J5 DB15_Female_HighDensity, J81 Conn_02x07_Counter_Clockwise, U2 FD8288T (DRV8300), U30 MCP2551-I-SN, U31 CPDT-12V, U80 STM32F103CBTx, U81 ABM3B-8.000MHZ

Commit message: initial copy from goldESC
Other:
- sheet GE-Fets-A renamed IE-Fets-A
- sheet GE-Fets-B renamed IE-Fets-B
- sheet GE-Fets-C renamed IE-Fets-C
- sheet GE-Regs renamed IE-Regs
- sheet IE-Fets-A: file GE-Fets.kicad_sch -> IE-Fets.kicad_sch
- sheet IE-Fets-B: file GE-Fets.kicad_sch -> IE-Fets.kicad_sch
- sheet IE-Fets-C: file GE-Fets.kicad_sch -> IE-Fets.kicad_sch
- sheet IE-Regs: file GE-Regs.kicad_sch -> IE-Regs.kicad_sch

Commit message: kicad V8
Parts:
- removed J5: DB15_Female_HighDensity, Connector_Dsub:DSUB-15-HD_Female_Horizontal_P2.29x1.98mm_EdgePinOffset3.03mm_Housed_MountingHolesOffset4.94mm, symbol Connector:DB15_Female_HighDensity
- added C11: 10nF, 6.3V, Capacitor_SMD:C_0402_1005Metric, symbol Device:C
- added C12: 22pF, Capacitor_SMD:C_0402_1005Metric, symbol Device:C
- added C13: 2.2uF, 6.3V, Capacitor_SMD:C_0402_1005Metric, symbol Device:C
- added C14: 2.2uF, 10V, Capacitor_SMD:C_0402_1005Metric, symbol Device:C
- added C2, C3: 330uF, AlfredoFootprints:Cap_THT_LowESR_330uF, symbol Device:C_Polarized
- added C8: 2.2uF, 50V, Capacitor_SMD:C_0603_1608Metric, symbol Device:C
- added C9: 100nF, Capacitor_SMD:C_0402_1005Metric, symbol Device:C
- added J2: Vin, AlfredoFootprints:GE_PwrPad1, symbol Connector_Generic:Conn_01x01
- added J3: Gnd, AlfredoFootprints:GE_PwrPad1, symbol Connector_Generic:Conn_01x01
- added L1: 4.7uH, Inductor_SMD:L_1210_3225Metric, symbol Device:L
- added R2: 100K, Resistor_SMD:R_0402_1005Metric, symbol Device:R
- added R3: 13K, Resistor_SMD:R_0402_1005Metric, symbol Device:R
- added U1: SY8113BADC, Package_TO_SOT_SMD:TSOT-23-6, symbol NoU265:SY8113BADC
- added U3: SPX3819M5-L-3-3, Package_TO_SOT_SMD:SOT-23-5, symbol Regulator_Linear:SPX3819M5-L-3-3
Connections:
- net +3V3: now also C13.2, U3.5 (OUT)
- net +5V: now also C12.2, C14.2, L1.2, R2.1, U3.1 (IN), U3.3 (EN)
- net GND: now also C11.1, C13.1, C14.1, C2.2, C3.2, C8.1, J3.1 (Pin_1), R3.2, U1.2 (GND), U3.2 (GND)
- net VDD: now also C2.1, C3.1, C8.2, J2.1 (Pin_1), U1.4 (EN), U1.5 (IN)
- new net: C9.1, L1.1, U1.6 (LX)
- new net: C9.2, U1.1 (BS)
- new net: C11.2, U3.4 (BP)
- new net: C12.1, R2.2, R3.1, U1.3 (FB)
Other:
- removed sheet IE-Regs
- note added: "330uF 16V Panasonic Low Impedance"

Commit message: updated with g431 info
Parts:
- removed C2, C3: 330uF, AlfredoFootprints:Cap_THT_LowESR_330uF, symbol Device:C_Polarized
- removed C80: 100nF, Capacitor_SMD:C_0402_1005Metric, symbol Device:C
- removed C81, C82, C83, C84: 2.2uF, 10V, Capacitor_SMD:C_0402_1005Metric, symbol Device:C
- removed C88, C89: 15pF, Capacitor_SMD:C_0402_1005Metric, symbol Device:C_Small
- removed J2: Vin, AlfredoFootprints:GE_PwrPad1, symbol Connector_Generic:Conn_01x01
- removed J3: Gnd, AlfredoFootprints:GE_PwrPad1, symbol Connector_Generic:Conn_01x01
- removed J81: Conn_02x07_Counter_Clockwise, AlfredoFootprints:Connector_2x05_P1.27mm_IDC, symbol Connector_Generic:Conn_02x05_Odd_Even
- removed R80: 10K, Resistor_SMD:R_0402_1005Metric, symbol Device:R
- removed TP80: TestPoint, AlfredoFootprints:GE_TestPoint_Loop, symbol Connector:TestPoint
- removed U80: STM32F103CBTx, Package_QFP:LQFP-48_7x7mm_P0.5mm, symbol MCU_ST_STM32F1:STM32F103C8Tx
- removed U81: ABM3B-8.000MHZ, Crystal:Crystal_SMD_5032-4Pin_5.0x3.2mm, symbol Device:Crystal_GND24
- added C15, C16: 15pF, Capacitor_SMD:C_0402_1005Metric, symbol Device:C_Small
- added C17: 100nF, Capacitor_SMD:C_0402_1005Metric, symbol Device:C
- added C18, C19: ~, Capacitor_SMD:CP_Elec_6.3x7.7, symbol Device:C_Polarized
- added C20, C21, C22, C23: 2.2uF, 10V, Capacitor_SMD:C_0402_1005Metric, symbol Device:C
- added D7: Z5V6, AlfredoFootprints:D_SOD-323, symbol Diode:ZMMxx
- added H1, H2, H3, H4: MountingHole, AlfredoFootprints:TGD_MountingHole, symbol Mechanical:MountingHole
- added J5: Conn_01x06, Connector_JST:JST_PH_B6B-PH-K_1x06_P2.00mm_Vertical, symbol Connector_Generic:Conn_01x06
- added J7: Screw_Terminal_01x02, AlfredoFootprints:TerminalBlock_Ningbo_2P_5mm, symbol Connector:Screw_Terminal_01x02
- added Q7: AO3401A, AlfredoFootprints:SOT-23-small, symbol Transistor_FET:AO3401A
- added R5, R6: 10K, Resistor_SMD:R_0402_1005Metric, symbol Device:R
- added R8: 1K, Resistor_SMD:R_0402_1005Metric, symbol Device:R
- added SW1: reset, AlfredoFootprints:Button_SKRKAEE020, symbol Switch:SW_Push
- added TP1: TestPoint, AlfredoFootprints:GE_TestPoint_Loop, symbol Connector:TestPoint
- added U7: STM32G431CBUx, Package_DFN_QFN:QFN-48-1EP_7x7mm_P0.5mm_EP5.6x5.6mm, symbol MCU_ST_STM32G4:STM32G431CBUx
- added U8: ABM3B-8.000MHZ, Crystal:Crystal_SMD_5032-4Pin_5.0x3.2mm, symbol Device:Crystal_GND24
- renumbered C8 to C800, C9 to C900, R2 to R200, R3 to R300
Connections:
- net +3V3: now also C20.1, C21.1, C22.1, C23.1, R8.2, U7.1 (VBAT), U7.21 (VDDA), U7.23 (VDD), U7.35 (VDD), U7.48 (VDD)
- net +5V: now also J5.6 (Pin_6)
- net GND: now also C15.1, C16.1, C17.2, C18.2, C19.2, C20.2, C21.2, C22.2, C23.2, J5.1 (Pin_1), J7.2 (Pin_2), R5.2, R6.2, SW1.2, U7.49 (VSS), U8.2, U8.4
- net VDD: now also C18.1, C19.1, D7.1 (K), Q7.2 (S)
- new net: R6.1, TP1.1, U7.46 (PB8)
- new net: D7.2 (A), Q7.1 (G), R5.1
- new net: C15.2, U7.5 (PF0), U8.1
- new net: C16.2, U7.6 (PF1), U8.3
- new net: J7.1 (Pin_1), Q7.3 (D)
- new net ENC_A: J5.3 (Pin_3)
- new net ENC_B: J5.4 (Pin_4)
- new net ENC_C: J5.5 (Pin_5)
- new net S2_EN: C17.1, R8.1, SW1.1, U7.7 (PG10)
- new net TEMP_A: J5.2 (Pin_2)
- no-connect marks 9 -> 2
Other:
- added sheet LORA (ExpressLRS-RX.kicad_sch)
- note added: "BLDC control: - 2 motors - open loop - sensorless - FOC DC control: - 3 motors Stepper motor: - 1 motor Wireless: - Lora - Meshtastic Charging: - 2 cell lipo - source from wall - source from solar IO: - qwiic - usb-c prog - Encoders Strech goal: - Express LRS - Drone - CAN"
- note added: "TODO: - Order JLC global source ASAP - test the current/voltage measuring circuit I already have - fiugre out micropython USB bootloader -switch to smaller pkg drv"

Commit message: push before removing bldc1 external opAmps
Parts:
- removed J30: CanOut, AlfredoFootprints:GE_SigPad_1x02, symbol Connector:Screw_Terminal_01x02
- removed J4: GND, AlfredoFootprints:GE_PwrPad1, symbol Connector_Generic:Conn_01x01
- removed R32: 51K, Resistor_SMD:R_0402_1005Metric, symbol Device:R
- removed R4: 2K, Resistor_SMD:R_0402_1005Metric, symbol Device:R
- removed R7: 1K, Resistor_SMD:R_0402_1005Metric, symbol Device:R
- removed R84, R85: 200R, Resistor_SMD:R_0402_1005Metric, symbol Device:R
- removed U30: MCP2551-I-SN, Package_SO:SOIC-8_3.9x4.9mm_P1.27mm, symbol Interface_CAN_LIN:MCP2551-I-SN
- removed U31: CPDT-12V, Package_TO_SOT_SMD:SOT-23, symbol AlfredoSymbols:CPDT-12V
- added C24, C25: 390pF, Capacitor_SMD:C_0402_1005Metric, symbol Device:C
- added C26: 100nF, 50V, Capacitor_SMD:C_0402_1005Metric, symbol Device:C
- added C27, C28, C32: 100nF, Capacitor_SMD:C_0402_1005Metric, symbol Device:C
- added C29: 250nF, Capacitor_THT:C_Rect_L9.0mm_W4.0mm_P7.50mm_MKT, symbol Device:C
- added C30, C31: 15nF, Capacitor_SMD:C_0402_1005Metric, symbol Device:C
- added C33, C34: 10uF,50V, Capacitor_SMD:C_1206_3216Metric, symbol Device:C
- added C35, C36: 2.2uF, Capacitor_SMD:C_0603_1608Metric, symbol Device:C
- added C37: 10uF,50V, Capacitor_SMD:C_1206_3216Metric, symbol Device:C_Small
- added C38, C39, C40: 1uF, Capacitor_SMD:C_0402_1005Metric, symbol Device:C_Small
- added D10: LED_Green, LED_SMD:LED_0603_1608Metric, symbol Device:LED
- added D11: ESDA6V1L, Package_TO_SOT_SMD:SOT-23-3, symbol Power_Protection:ESDA5V3L
- added D13: ESDA25P35-1U1M, AlfredoFootprints:DFN1610-2, symbol Device:D_Zener
- added D14, D8: 1N5819, AlfredoFootprints:D_SOD-323, symbol Device:D_Zener
- added D15, D16, D17: SDM20U40-7, Diode_SMD:D_SOD-523, symbol Diode:US1M
- added D9: LED_Red, LED_SMD:LED_0603_1608Metric, symbol Device:LED
- added J1: JST SR/SZ, AlfredoFootprints:JST_SH_1x06_Vertical, symbol Connector_Generic:Conn_01x06
- added J10: VIN_BARREL, AlfredoFootprints:DC-005C_1, symbol Connector:Barrel_Jack
- added J11: Barrel_Jack, AlfredoFootprints:DC-005C_1, symbol Connector:Barrel_Jack
- added J2, J3, J4: Screw_Terminal_01x02, AlfredoFootprints:TerminalBlock_Ningbo_2P_5mm, symbol Connector:Screw_Terminal_01x02
- added J6: Wireless Coil, AlfredoFootprints:TerminalBlock_Ningbo_2P_5mm, symbol Connector:Screw_Terminal_01x02
- added J8: Conn_01x06, Connector_JST:JST_PH_B6B-PH-K_1x06_P2.00mm_Vertical, symbol Connector_Generic:Conn_01x06
- added JP1: Qi_Enable, Connector_PinSocket_2.54mm:PinSocket_1x02_P2.54mm_Vertical, symbol Jumper:Jumper_2_Open
- added JP2: VRAW to VCC, Connector_PinSocket_2.54mm:PinSocket_1x02_P2.54mm_Vertical, symbol Jumper:Jumper_2_Open
- added JP3: Fets_Enable1, Connector_PinSocket_2.54mm:PinSocket_1x02_P2.54mm_Vertical, symbol Jumper:Jumper_2_Open
- added JP4: Fets_Enable2, Connector_PinSocket_2.54mm:PinSocket_1x02_P2.54mm_Vertical, symbol Jumper:Jumper_2_Open
- added R20, R26, R27: 100K, Resistor_SMD:R_0402_1005Metric, symbol Device:R
- added R28, R29: 1K, Resistor_SMD:R_0402_1005Metric, symbol Device:R
- added R33: 20mR, Resistor_SMD:R_0603_1608Metric, symbol Device:R
- added R34: 10K, Resistor_SMD:R_0402_1005Metric, symbol Device:R
- added R35: 33K, Resistor_SMD:R_0402_1005Metric, symbol Device:R
- added R9: 3K3, Resistor_SMD:R_0402_1005Metric, symbol Device:R
- added TP10, TP5: TP_CC2, AlfredoFootprints:GE_TestPoint_Loop, symbol Connector:TestPoint
- added TP2: TP_DM, AlfredoFootprints:GE_TestPoint_Loop, symbol Connector:TestPoint
- added TP3: TP_DP, AlfredoFootprints:GE_TestPoint_Loop, symbol Connector:TestPoint
- added TP4: TP_DEBUG, AlfredoFootprints:GE_TestPoint_Loop, symbol Connector:TestPoint
- added TP6, TP9: TP_CC1, AlfredoFootprints:GE_TestPoint_Loop, symbol Connector:TestPoint
- added U10: USBLC6-2P6, Package_TO_SOT_SMD:SOT-666, symbol Power_Protection:USBLC6-2P6
- added U11: IP6826, Package_DFN_QFN:QFN-32-1EP_5x5mm_P0.5mm_EP3.7x3.7mm, symbol AlfredoSymbols:IP6826
- added U12: FD8288T (DRV8300), Package_SO:TSSOP-20_4.4x6.5mm_P0.65mm, symbol AlfredoSymbols:DRV8300NIPWR
- added U13: Qwiic1, Connector_JST:JST_SH_BM04B-SRSS-TB_1x04-1MP_P1.00mm_Vertical, symbol AlfredoSymbols:QwiicConnector
- added U9: USB_C_Receptacle, AlfredoFootprints:USB_TYPE-C-31-M-12, symbol Connector:USB_C_Receptacle
- C18, C19: value ~ -> 220uF
- D83, D84: footprint LED_SMD:LED_0805_2012Metric -> LED_SMD:LED_0603_1608Metric
- J7: value Screw_Terminal_01x02 -> VIN_TERMINAL
- R30: value 5.6K -> 1K; LCSC C25908 -> C11702
- R31: value 10K -> 1K; LCSC C25744 -> C11702
Connections:
- net +3V3: now also J1.4 (Pin_4), U13.2 (3V3)
- net +5V: now also C37.1, D15.2 (A), D16.2 (A), D17.2 (A), J8.6 (Pin_6), U12.7 (GVDD)
- net GND: now also U7.13 (PA5), U7.19 (PB2), U7.9 (PA1), C24.2, C25.2, C26.2, C35.1, C36.1, C37.2, D10.1 (K), D11.3 (A), D13.2 (A), D9.1 (K), J1.1 (Pin_1), J10.2, J11.2, J8.1 (Pin_1), R26.2, R27.2, R33.1, U10.2 (GND), U11.1 (GND), U11.2 (IGND), U11.32 (AGND), U12.8 (GND), U13.1 (GND), U9.A1 (GND), U9.A12 (GND), U9.B1 (GND), U9.B12 (GND); no longer R31.2
- net SCL: now also U13.4 (SCL)
- net SDA: now also U13.3 (SDA)
- net SWCLK: now also U7.37 (PA14)
- net SWDIO: now also U7.36 (PA13)
- net at D84.2 (A): now also R31.2
- net VIN: now reaches J7.1 (Pin_1), Q7.3 (D)
- net VIN: now also J10.1
- net at D83.2 (A): now also R30.2
- net sCUR_A2_OUT: now reaches U7.10 (PA2)
- net sCUR_A2_OUT: now also J8.3 (Pin_3)
- net sCUR_A2+: now reaches U7.11 (PA3)
- net sVLT_A2: now reaches U7.12 (PA4)
- net sCUR_B2_OUT: now reaches U7.14 (PA6)
- net sCUR_B2_OUT: now also J8.4 (Pin_4)
- net sCUR_B2+: now reaches U7.15 (PA7)
- net sCUR_C2+: now reaches U7.16 (PC4)
- net sVLT_B2: now reaches U7.17 (PB0)
- net sCUR_C2_OUT: now reaches U7.18 (PB1)
- net sCUR_C2_OUT: now also J8.5 (Pin_5)
- net sVLT_C2: now reaches U7.24 (PB11)
- net USB_D-: now reaches U7.33 (PA11)
- net USB_D-: now also U10.3 (I/O2), U10.4 (I/O2), U9.A7 (D-), U9.B7 (D-)
- net USB_D+: now reaches U7.34 (PA12)
- net USB_D+: now also U10.1 (I/O1), U10.6 (I/O1), U9.A6 (D+), U9.B6 (D+)
- net CC2: now reaches U7.42 (PB4)
- net CC2: now also C24.1, D11.2 (K), TP10.1, U9.B5 (CC2)
- net CC1: now reaches U7.44 (PB6)
- net CC1: now also C25.1, D11.1 (K), TP9.1, U9.A5 (CC1)
- net CAN_RX: no longer names the net of R31.1
- net CAN_RX: no longer R30.2
- net ENC_A renamed ENC_A1
- net ENC_A1: now also J1.3 (Pin_3)
- net ENC_B renamed ENC_B1
- net ENC_B1: now also J1.2 (Pin_2)
- net ENC_C renamed ENC_C1
- net INHA renamed INHA_1
- net INHB renamed INHB_1
- net INHC renamed INHC_1
- net INLA renamed INLA_1
- net INLB renamed INLB_1
- net INLC renamed INLC_1
- net TEMP_A renamed TEMP_1
- net VDD renamed VRAW
- net VRAW: now also JP1.1 (A), JP2.2 (B), JP3.1 (A), JP4.1 (A); no longer C800.2, U1.4 (EN), U1.5 (IN)
- net sVLT_VDD renamed sVLT_VRAW
- new net: C27.1, U11.19 (BST1)
- new net: C27.2, C29.2, U11.20 (LX1), U11.21 (LX1)
- new net: TP2.1, U11.28 (DM)
- new net: C38.1, D15.1 (K), U12.20 (BSTA)
- new net: C40.1, D17.1 (K), U12.14 (BSTC)
- new net: D14.1 (K), R20.1, R9.1
- new net: TP5.1, U11.9 (CC2)
- new net: C32.2, C33.2, C34.2, JP1.2 (B), U11.26 (VIN), U11.27 (VIN)
- new net: D10.2 (A), R29.1
- new net: TP4.1, U11.10 (DEBUG)
- new net: R26.1, U11.11 (NTC)
- new net: R27.1, U11.12 (LOSS_THR)
- new net: R29.2, U11.13 (LED1)
- new net: R28.2, U11.16 (LED2)
- new net: C28.2, J6.1 (Pin_1), U11.22 (LX2), U11.23 (LX2)
- new net: C28.1, U11.24 (BST2)
- new net: TP3.1, U11.29 (DP)
- new net: C35.2, U11.4 (VCC)
- new net: TP6.1, U11.8 (CC1)
- new net: C39.1, D16.1 (K), U12.17 (BSTB)
- new net: C30.1, C31.2, R35.1, R9.2
- new net: C31.1, R34.2, R35.2
- new net: D9.2 (A), R28.1
- new net: C29.1, D14.2 (A), J6.2 (Pin_2)
- new net IE-FETS-NoOp-A/GHx: U12.19 (GHA)
- new net IE-FETS-NoOp-A/GLx: U12.11 (GLA)
- new net IE-FETS-NoOp-A/SHx: C38.2, U12.18 (SHA)
- new net IE-FETS-NoOp-A/VFET: JP4.2 (B)
- new net IE-FETS-NoOp-A/VOUT: J1.6 (Pin_6), J3.1 (Pin_1)
- new net IE-FETS-NoOp-B/GHx: U12.16 (GHB)
- new net IE-FETS-NoOp-B/GLx: U12.10 (GLB)
- new net IE-FETS-NoOp-B/SHx: C39.2, U12.15 (SHB)
- new net IE-FETS-NoOp-B/VOUT: J4.2 (Pin_2)
- new net IE-FETS-NoOp-C/GHx: U12.13 (GHC)
- new net IE-FETS-NoOp-C/GLx: U12.9 (GLC)
- new net IE-FETS-NoOp-C/SHx: C40.2, U12.12 (SHC)
- new net IE-FETS-NoOp-C/VOUT: J4.1 (Pin_1)
- new net IE-Fets-A/VFET: JP3.2 (B)
- new net IE-Fets-A/VOUT: J11.1, J2.2 (Pin_2)
- new net IE-Fets-B/VOUT: J2.1 (Pin_1)
- new net IE-Fets-C/VOUT: J1.5 (Pin_5), J3.2 (Pin_2)
- new net INHA_2: U12.1 (INHA)
- new net INHB_2: U12.2 (INHB)
- new net INHC_2: U12.3 (INHC)
- new net INLA_2: U12.4 (INLA)
- new net INLB_2: U12.5 (INLB)
- new net INLC_2: U12.6 (INLC)
- new net PGND: C32.1, C33.1, C34.1, R33.2, U11.3 (ISENSE), U11.33 (G_PAD), U11.5 (PGND)
- new net TEMP_2: J8.2 (Pin_2)
- new net VCC: C800.2, D8.1 (K), JP2.1 (A), U1.4 (EN), U1.5 (IN)
- new net V_DECODE: C30.2, U11.18 (V_DECODE)
- new net V_DETECT: C36.2, R20.2, R34.1, U11.30 (VDET)
- new net V_USB: C26.1, D13.1 (K), D8.2 (A), U9.A4 (VBUS), U9.A9 (VBUS), U9.B4 (VBUS), U9.B9 (VBUS)
- no-connect marks 2 -> 20
Other:
- removed sheet LORA
- added sheet IE-FETS-NoOp-A (IE-FETS-NoOp.kicad_sch)
- added sheet IE-FETS-NoOp-B (IE-FETS-NoOp.kicad_sch)
- added sheet IE-FETS-NoOp-C (IE-FETS-NoOp.kicad_sch)
- sheet IE-Fets-A ports: added VFET, VOUT; removed none
- sheet IE-Fets-B ports: added VFET, VOUT; removed none
- sheet IE-Fets-C ports: added VFET, VOUT; removed none
- note added: "Vin max = 18V TODO: look into ideal diodes () look into PTC fuses (MF-MSMF050-2) done:"
- note removed: "ADC12_IN0 ADC12_IN1 ADC12_IN2 ADC12_IN3 ADC12_IN4 ADC12_IN5 ADC12_IN6 ADC12_IN7"
- note removed: "ADC12_IN8 ADC12_IN9"
- note removed: "T1_CH1 T1_CH2 T1_CH3"
- note removed: "T1_CH1N T1_CH2N T1_CH3N"
- note removed: "Vin max = 18V TODO: Fix current sense precision issue done: switch A and C phase parts switch to LDR 3v3 reg? add TVS diodes change connector new leds change boot0 ckt to allow usb bootloader rethink C10? rethink bulk caps? rething C1-C3? change 0603s to 0402s do I really need sVLT_x? (yes) pick smaller 3V3 Z_diodes"
- moved on the sheet: C10, C11, C12, C13, C14, C4, C42, C5, C6, C800, C900, D4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

Commit message: push for 8/8 order
Parts:
- removed C23: 2.2uF, 10V, Capacitor_SMD:C_0402_1005Metric, symbol Device:C
- removed JP4: Fets_Enable2, Connector_PinSocket_2.54mm:PinSocket_1x02_P2.54mm_Vertical, symbol Jumper:Jumper_2_Open
- removed R6: 10K, Resistor_SMD:R_0402_1005Metric, symbol Device:R
- removed TP83, TP84: TestPoint, AlfredoFootprints:GE_TestPoint_Loop, symbol Connector:TestPoint
- added C7, C8, C9: 0.1uF, Capacitor_SMD:C_0402_1005Metric, symbol Device:C
- added FB1: BLM15BX601SN1D, Inductor_SMD:L_0402_1005Metric, symbol Device:FerriteBead
- added J12, J9: JST SR/SZ, AlfredoFootprints:JST_SH_1x06_Vertical, symbol Connector_Generic:Conn_01x06
- added R2: 1K, Resistor_SMD:R_0402_1005Metric, symbol Device:R
- added TP7: SWDIO, AlfredoFootprints:GE_TestPoint_Loop, symbol Connector:TestPoint
- added TP8: SWCLK, AlfredoFootprints:GE_TestPoint_Loop, symbol Connector:TestPoint
- C20: value 2.2uF, 10V -> 2.2uF
- C21: value 2.2uF, 10V -> 1uF; LCSC C77002 -> (none)
- C22: value 2.2uF, 10V -> 10nF; LCSC C77002 -> (none)
- D83: value LED_Red -> LED_Blue
- L1: LCSC C86070 -> C98354
- TP1: value TestPoint -> GND
- U8: footprint Crystal:Crystal_SMD_5032-4Pin_5.0x3.2mm -> Crystal:Crystal_SMD_3225-4Pin_3.2x2.5mm; LCSC C276420 -> C400090
Connections:
- net IE-Fets-A/VFET is gone; now on net IE-FETS-NoOp-A/VFET: JP3.2 (B)
- net SWCLK is gone; now on net SDA: U7.37 (PA14)
- net SWDIO is gone; now on net SCL: U7.36 (PA13)
- net +3V3: now also R30.1, C7.1, C8.1, C9.1, FB1.1, J12.4 (Pin_4), J9.4 (Pin_4); no longer C21.1, C22.1, U7.21 (VDDA)
- net CC1: now also D11.2 (K); no longer D11.1 (K)
- net CC2: now also D11.1 (K); no longer D11.2 (K)
- net ENC_A1: now also U7.29 (PC6)
- net ENC_B1: now also U7.3 (PC14)
- net ENC_C1: now also U7.4 (PC15), J9.2 (Pin_2)
- net GND: now also TP1.1, U7.11 (PA3), U7.22 (PB10), C7.2, C8.2, C9.2, J12.1 (Pin_1), J9.1 (Pin_1), R2.2; no longer U7.19 (PB2), U7.9 (PA1)
- net IE-FETS-NoOp-B/VOUT: now also J12.5 (Pin_5)
- net IE-FETS-NoOp-C/VOUT: now also J11.1, J12.6 (Pin_6)
- net IE-Fets-A/VOUT: now also J9.5 (Pin_5); no longer J11.1
- net IE-Fets-B/VOUT: now also J9.6 (Pin_6)
- net INHA_1: now also U7.47 (PB9)
- net INHA_2: now also U7.32 (PA10)
- net INHB_1: now also U7.46 (PB8), R2.1
- net INHB_2: now also U7.31 (PA9)
- net INHC_1: now also U7.38 (PA15)
- net INHC_2: now also U7.30 (PA8)
- net INLA_1: now also U7.43 (PB5)
- net INLA_2: now also U7.28 (PB15)
- net INLB_1: now also U7.40 (PC11)
- net INLB_2: now also U7.27 (PB14)
- net INLC_1: now also U7.39 (PC10)
- net INLC_2: now also U7.2 (PC13)
- net SCL: now also TP7.1
- net SDA: now also TP8.1
- net TEMP_1: now also U7.19 (PB2), J12.2 (Pin_2)
- net TEMP_2: now also U7.8 (PA0), J12.3 (Pin_3)
- net TEMP_FETS: now also U7.17 (PB0)
- net sCUR_A2+: now also U7.9 (PA1); no longer U7.11 (PA3)
- net sCUR_C2+: now also U7.26 (PB13); no longer U7.16 (PC4)
- net sVLT_B2: now also U7.16 (PC4); no longer U7.17 (PB0)
- net sVLT_VRAW: now also U7.25 (PB12)
- net STM_LED: now reaches R31.1
- net STM_LED: now also U7.41 (PB3)
- net at U7.20 (VREF+): now also C21.1, C22.1, U7.21 (VDDA), FB1.2
- net lone_dc_encoder_pin: now reaches U7.45 (PB7)
- net lone_dc_encoder_pin: now also J9.3 (Pin_3)
Other:
- sheet IE-Fets-A ports: added none; removed sCURx, sVLTx
- sheet IE-Fets-B ports: added none; removed sCURx, sVLTx
- sheet IE-Fets-C ports: added none; removed sCURx, sVLTx
- note added: "2.2uF for VDD35"
- note added: "ADC1_IN12"
- note added: "ADC1_IN3"
- note added: "ADC2_IN3"
- note added: "TODO: max VIN is 18V from buck converter (upgrade?) done: VREF inductor fix stm caps Breakout SW-debug"
- note removed: "330uF 16V Panasonic Low Impedance"
- note removed: "Vin max = 18V TODO: look into ideal diodes () look into PTC fuses (MF-MSMF050-2) done:"
- note removed: "for VDDA"
- moved on the sheet: C12, C14, C18, C19, C20, C24, C25, C26, C27, C28, C29, C30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

Commit message: first push for v2
Parts:
- added C23: 100nF, 50V, Capacitor_SMD:C_0402_1005Metric, symbol Device:C
- added SW2, SW3: boot, AlfredoFootprints:Button_SKRKAEE020, symbol Switch:SW_Push
- added U4: STM32G474RETx, Package_QFP:LQFP-64_10x10mm_P0.5mm, symbol MCU_ST_STM32G4:STM32G474RETx
- C10, C33, C34, C37: value 10uF,50V -> 10uF, 50V
- C13: value 2.2uF, 6.3V -> 2.2uF, 10V; LCSC C12530 -> C77002
- C15, C16: value 15pF -> 15pF, 50V
- C17, C42, C900: value 100nF -> 100nF, 50V
- C20: value 2.2uF -> 2.2uF, 10V
- C21: LCSC (none) -> C52923
- C22: value 10nF -> 10nF, 6.3V; LCSC (none) -> C15195
- C27, C28, C32: value 100nF -> 100nF, 50V; LCSC (none) -> C307331
- C29: value 250nF -> 250nF, 100V
- C35, C36: value 2.2uF -> 2.2uF, 50V
- C7, C8, C9: value 0.1uF -> 100nF, 50V; LCSC (none) -> C307331
Connections:
- net +3V3: now also C21.1, C22.1, FB1.2, C23.1, SW2.1, U4.1 (VBAT), U4.16 (VDD), U4.28 (VREF+), U4.29 (VDDA), U4.32 (VDD), U4.48 (VDD), U4.64 (VDD); no longer U7.1 (VBAT), U7.23 (VDD), U7.35 (VDD), U7.48 (VDD)
- net GND: now also C31.1, R34.2, R35.2, U4.15 (VSS), U4.27 (VSSA), U4.31 (VSS), U4.47 (VSS), U4.63 (VSS)
- net INHB_1: no longer R2.1, U7.46 (PB8)
- net at C15.2, U8.1: now also U4.5 (PF0); no longer U7.5 (PF0)
- net at C16.2, U8.3: now also U4.6 (PF1); no longer U7.6 (PF1)
- net S2_EN: no longer names the net of C17.1, R8.1, SW1.1
- net S2_EN: now also U4.7 (PG10); no longer U7.7 (PG10)
- new net: C23.2, R2.1, SW2.2, U4.40 (PC8)
- now unconnected: U7.20 (VREF+), U7.21 (VDDA)
Other:
- note added: "long term: - max VIN is 18V from buck converter (upgrade?) - test the current/voltage measuring circuit I already have - switch to smaller pkg drv V2 TODO - power rate indicator LEDs - mode buttons with indicator - change G432 to G474 - Boot button is actually rst (fix this) - add boot button for DFU - fix wireless charger - improve SWD interface? (or is 4 pin jst good?) - better test probes - cu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"
- note removed: "Ref-map: 1 -29 -> fets/driver 30-39 -> CAN 40-69 -> Regs 70-89 -> STM32"
- note removed: "TODO: - Order JLC global source ASAP - test the current/voltage measuring circuit I already have - fiugre out micropython USB bootloader -switch to smaller pkg drv"
- note removed: "TODO: max VIN is 18V from buck converter (upgrade?) done: VREF inductor fix stm caps Breakout SW-debug"
- moved on the sheet: C11, C12, C13, C14, C15, C16, C17, C18, C19, C21, C22, C800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
