File: I3ESC.kicad_sch (KiCad schematic)
At the start: 122 parts, among them J1 JST SR/SZ, J10 VIN_BARREL, J11 Barrel_Jack, J12 JST SR/SZ, J2 Screw_Terminal_01x02, J3 Screw_Terminal_01x02, J4 Screw_Terminal_01x02, J5 Conn_01x06, J6 Wireless Coil, J7 VIN_TERMINAL, J8 Conn_01x06, J9 JST SR/SZ, Q7 AO3401A, SW1 reset, SW2 boot, SW3 boot, U1 SY8113BADC, U10 USBLC6-2P6, U11 IP6826, U12 FD8288T (DRV8300), U13 Qwiic1, U2 FD8288T (DRV8300), U3 SPX3819M5-L-3-3, U4 STM32G474RETx, U7 STM32G431CBUx, U8 ABM3B-8.000MHZ, U9 USB_C_Receptacle

Commit message: big schematic push for stm32g474
Parts:
- removed D7: Z5V6, AlfredoFootprints:D_SOD-323, symbol Diode:ZMMxx
- removed Q7: AO3401A, AlfredoFootprints:SOT-23-small, symbol Transistor_FET:AO3401A
- removed U7: STM32G431CBUx, Package_DFN_QFN:QFN-48-1EP_7x7mm_P0.5mm_EP5.6x5.6mm, symbol MCU_ST_STM32G4:STM32G431CBUx
- added C45, C46: 100nF, 50V, Capacitor_SMD:C_0402_1005Metric, symbol Device:C
- added D7: LED_RED, LED_SMD:LED_0603_1608Metric, symbol Device:LED
- added R67: 1K, Resistor_SMD:R_0402_1005Metric, symbol Device:R
- added U5: Qwiic1, Connector_JST:JST_SH_BM04B-SRSS-TB_1x04-1MP_P1.00mm_Vertical, symbol AlfredoSymbols:QwiicConnector
- D42: footprint Diode_SMD:D_SOD-323_HandSoldering -> Diode_SMD:D_SOD-523; LCSC C75073 -> C2891760
- R5: value 10K -> 1K; LCSC C25744 -> C11702
- SW3: value boot -> user1
Connections:
- net INHA_1 is gone; now on net IN_H_1A: U2.1 (INHA)
- net INHA_2 is gone; now on net IN_H_2A: U12.1 (INHA)
- net INHB_1 is gone; now on net IN_H_1B: U2.2 (INHB)
- net INHB_2 is gone; now on net IN_H_2B: U12.2 (INHB)
- net INHC_1 is gone; now on net IN_H_1C: U2.3 (INHC)
- net INHC_2 is gone; now on net IN_H_2C: U12.3 (INHC)
- net INLA_1 is gone; now on net IN_L_1A: U2.4 (INLA)
- net INLB_1 is gone; now on net IN_L_1B: U2.5 (INLB)
- net INLB_2 is gone; now on net IN_L_2B: U12.5 (INLB)
- net INLC_1 is gone; now on net IN_L_1C: U2.6 (INLC)
- net INLC_2 is gone; now on net IN_L_2C: U12.6 (INLC)
- net STM_LED is gone; now on net STM_LED1: R31.1
- net TEMP_FETS is gone; now on net OPAMP3_VOUT: R40.2, R41.1
- net VIN is gone; now on net VRAW: J10.1, J7.1 (Pin_1)
- net +3V3: now also SW3.1, C46.1, U5.2 (3V3); no longer C23.1
- net CC1: now also U4.59 (PB6)
- net CC2: now also U4.57 (PB4)
- net GND: now also C23.2, C45.2, C46.2, D7.1 (K), R67.2, U5.1 (GND); no longer J11.2, R5.2
- net IE-FETS-2B/VOUT: now also J11.1
- net IE-FETS-2C/VOUT: now also J11.2; no longer J11.1
- net SCL: now also U4.51 (PA15); no longer TP7.1
- net SDA: now also U4.60 (PB7); no longer TP8.1
- net USB_D+: now also U4.46 (PA12)
- net USB_D-: now also U4.45 (PA11)
- net sVLT_VRAW: now also U4.12 (PA0)
- net BOOT: now reaches R2.1, SW2.2
- net BOOT: now also C23.1, U4.61 (PB8); no longer C23.2, U4.40 (PC8)
- net STM_LED2: now reaches R5.1
- net STM_LED2: now also U4.44 (PA10)
- net IN_H_1C: now reaches U4.10 (PC2)
- net IN_L_1C: now reaches U4.11 (PC3)
- net OPAMP1_V+: now reaches U4.13 (PA1)
- net OPAMP1_VOUT: now reaches U4.14 (PA2)
- net sVLT_1A: now reaches U4.17 (PA3)
- net sVLT_1B: now reaches U4.18 (PA4)
- net sVLT_1C: now reaches U4.19 (PA5)
- net ENC_1A: now reaches U4.2 (PC13)
- net OPAMP2_VOUT: now reaches U4.20 (PA6)
- net OPAMP2_V+: now reaches U4.21 (PA7)
- net IN_H_2A: now reaches U4.22 (PC4)
- net IN_H_2B: now reaches U4.23 (PC5)
- net OPAMP3_V+: now reaches U4.24 (PB0)
- net OPAMP3_VOUT: now reaches U4.25 (PB1)
- net sVLT_2B: now reaches U4.26 (PB2)
- net ENC_1B: now reaches U4.3 (PC14)
- net ENC_2C: now reaches U4.30 (PB10)
- net OPAMP6_VOUT: now reaches U4.33 (PB11)
- net OPAMP4_VOUT: now reaches U4.34 (PB12)
- net OPAMP4_V+: now reaches U4.35 (PB13)
- net OPAMP5_V+: now reaches U4.36 (PB14)
- net IN_H_1A: now reaches U4.37 (PB15)
- net IN_H_2C: now reaches U4.38 (PC6)
- net STM_LED1: now reaches U4.39 (PC7)
- net ENC_1C: now reaches U4.4 (PC15)
- net IN_L_2B: now reaches U4.41 (PC9)
- net OPAMP5_VOUT: now reaches U4.42 (PA8)
- net sVLT_2A: now reaches U4.43 (PA9)
- net SWDIO: now reaches U4.49 (PA13)
- net SWDIO: now also TP7.1, U5.4 (SCL)
- net SWCLK: now reaches U4.50 (PA14)
- net SWCLK: now also TP8.1, U5.3 (SDA)
- net IN_L_2C: now reaches U4.52 (PC10)
- net IN_L_1A: now reaches U4.53 (PC11)
- net USER1: now reaches U4.54 (PC12)
- net USER1: now also SW3.2, C45.1, R67.1
- net ENC_2A: now reaches U4.56 (PB3)
- net ENC_2B: now reaches U4.58 (PB5)
- net IN_L_1B: now reaches U4.62 (PB9)
- net sVLT_2C: now reaches U4.8 (PC0)
- net IN_H_1B: now reaches U4.9 (PC1)
- net IE-FETS-2A/VFET renamed IE-FETS-1A/VFET
- net IE-Fets-A/GHx renamed IE-FETS-1A/GHx
- net IE-Fets-A/GLx renamed IE-FETS-1A/GLx
- net IE-Fets-A/SHx renamed IE-FETS-1A/SHx
- net IE-Fets-A/VOUT renamed IE-FETS-1A/VOUT
- net IE-Fets-B/GHx renamed IE-FETS-1B/GHx
- net IE-Fets-B/GLx renamed IE-FETS-1B/GLx
- net IE-Fets-B/SHx renamed IE-FETS-1B/SHx
- net IE-Fets-B/VOUT renamed IE-FETS-1B/VOUT
- net IE-Fets-C/GHx renamed IE-FETS-1C/GHx
- net IE-Fets-C/GLx renamed IE-FETS-1C/GLx
- net IE-Fets-C/SHx renamed IE-FETS-1C/SHx
- net IE-Fets-C/VOUT renamed IE-FETS-1C/VOUT
- net INLA_2 renamed IN_L_2A
- net IN_L_2A: now also U4.40 (PC8)
- new net: D7.2 (A), R5.2
Other:
- sheet IE-FETS-NoOp-A renamed IE-FETS-2A
- sheet IE-FETS-NoOp-B renamed IE-FETS-2B
- sheet IE-FETS-NoOp-C renamed IE-FETS-2C
- removed sheet IE-Fets-A
- removed sheet IE-Fets-B
- removed sheet IE-Fets-C
- added sheet IE-FETS-1A (IE-FETS.kicad_sch)
- added sheet IE-FETS-1B (IE-FETS.kicad_sch)
- added sheet IE-FETS-1C (IE-FETS.kicad_sch)
- sheet IE-FETS-2A: file IE-FETS-NoOp.kicad_sch -> IE-FETS.kicad_sch
- sheet IE-FETS-2B: file IE-FETS-NoOp.kicad_sch -> IE-FETS.kicad_sch
- sheet IE-FETS-2C: file IE-FETS-NoOp.kicad_sch -> IE-FETS.kicad_sch
- note added: "2.2uF for VDD32"
- note added: "long term: - max VIN is 18V from buck converter (upgrade?) - switch to smaller pkg drv SIG TODO: - power rate indicator LEDs - mode buttons with indicator - fix wireless charger - better test probes - current sns for wireless coil? - pick new SWD/I2C pins POWER TODO: - Bulk up RPP fet - do I need a power switch? - find power diode for D8 done: - improve SWD interface? (or is 4 pin jst good?) - ch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"
- note removed: "2.2uF for VDD35"
- note removed: "ADC1_IN12"
- note removed: "ADC1_IN3"
- note removed: "ADC2_IN3"
- note removed: "long term: - max VIN is 18V from buck converter (upgrade?) - test the current/voltage measuring circuit I already have - switch to smaller pkg drv V2 TODO - power rate indicator LEDs - mode buttons with indicator - change G432 to G474 - Boot button is actually rst (fix this) - add boot button for DFU - fix wireless charger - improve SWD interface? (or is 4 pin jst good?) - better test probes - cu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"
- moved on the sheet: C15, C16, C17, C18, C19, C20, C21, C22, C7, C8, C9, FB1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

Commit message: huge layout progress
Parts:
- removed C17: 100nF, 50V, Capacitor_SMD:C_0402_1005Metric, symbol Device:C
- removed C19: 220uF, Capacitor_SMD:CP_Elec_6.3x7.7, symbol Device:C_Polarized
- removed JP3: Fets_Enable1, Connector_PinSocket_2.54mm:PinSocket_1x02_P2.54mm_Vertical, symbol Jumper:Jumper_2_Open
- removed SW1: reset, AlfredoFootprints:Button_SKRKAEE020, symbol Switch:SW_Push
- removed TP10: TP_CC2, AlfredoFootprints:GE_TestPoint_Loop, symbol Connector:TestPoint
- removed TP3: TP_DP, AlfredoFootprints:GE_TestPoint_Loop, symbol Connector:TestPoint
- removed TP7: SWDIO, AlfredoFootprints:GE_TestPoint_Loop, symbol Connector:TestPoint
- removed TP8: SWCLK, AlfredoFootprints:GE_TestPoint_Loop, symbol Connector:TestPoint
- removed TP9: TP_CC1, AlfredoFootprints:GE_TestPoint_Loop, symbol Connector:TestPoint
- removed U13: Qwiic1, Connector_JST:JST_SH_BM04B-SRSS-TB_1x04-1MP_P1.00mm_Vertical, symbol AlfredoSymbols:QwiicConnector
- added J13: Conn_01x04, Connector_PinHeader_2.54mm:PinHeader_1x04_P2.54mm_Vertical, symbol Connector_Generic:Conn_01x04
- added JP4: Qi_D-, Connector_PinSocket_2.54mm:PinSocket_1x02_P2.54mm_Vertical, symbol Jumper:Jumper_2_Open
- added JP5: Qi_D+, Connector_PinSocket_2.54mm:PinSocket_1x02_P2.54mm_Vertical, symbol Jumper:Jumper_2_Open
- added JP6: Qi_CC2, Connector_PinSocket_2.54mm:PinSocket_1x02_P2.54mm_Vertical, symbol Jumper:Jumper_2_Open
- added JP7: Qi_CC1, Connector_PinSocket_2.54mm:PinSocket_1x02_P2.54mm_Vertical, symbol Jumper:Jumper_2_Open
- added U6: USB_C_Receptacle, AlfredoFootprints:USB_TYPE-C-31-M-12, symbol Connector:USB_C_Receptacle
- JP2: value VRAW to VCC -> VCC-bypass; footprint Connector_PinSocket_2.54mm:PinSocket_1x02_P2.54mm_Vertical -> AlfredoFootprints:SolderJumper-2-Small
- SW2: value boot -> boot-red; footprint AlfredoFootprints:Button_SKRKAEE020 -> AlfredoFootprints:button-3.6x6mm; LCSC C115357 -> C255802
- SW3: value user1 -> user1-white; footprint AlfredoFootprints:Button_SKRKAEE020 -> AlfredoFootprints:button-3.6x6mm; LCSC C115357 -> C455236
- TP2: value TP_DM -> QI_PGND
Connections:
- net ENC_A1 is gone; now on net ENC_1C: J1.3 (Pin_3), J5.3 (Pin_3)
- net lone_dc_encoder_pin is gone; now on net ENC_1A: J9.3 (Pin_3)
- net sCUR_A2_OUT is gone; now on net ENC_2C: J8.3 (Pin_3)
- net sCUR_B2_OUT is gone; now on net ENC_2B: J8.4 (Pin_4)
- net sCUR_C2_OUT is gone; now on net ENC_2A: J8.5 (Pin_5)
- net +3V3: now also R40.1, J13.4 (Pin_4); no longer C21.1, C22.1, FB1.2, U4.28 (VREF+), U4.29 (VDDA)
- net +5V: no longer R40.1
- net ENC_1A: now also J5.5 (Pin_5)
- net ENC_1B: now also J5.4 (Pin_4), J9.2 (Pin_2)
- net ENC_2A: now also J1.2 (Pin_2)
- net ENC_2B: now also J12.3 (Pin_3)
- net ENC_2C: now also J12.2 (Pin_2)
- net GND: now also J13.1 (Pin_1), U6.A1 (GND), U6.A12 (GND), U6.B1 (GND), U6.B12 (GND)
- net PGND: now also TP2.1
- net SCL: now also J13.3 (Pin_3)
- net SDA: now also J13.2 (Pin_2)
- net STM_LED1: now also U4.44 (PA10); no longer U4.39 (PC7)
- net STM_LED2: now also U4.39 (PC7); no longer U4.44 (PA10)
- net TEMP_1: no longer J12.2 (Pin_2)
- net TEMP_2: no longer J12.3 (Pin_3)
- net VCC: now also C18.1, J10.1, J7.1 (Pin_1), R43.2
- net V_USB: now also JP2.2 (B)
- net at U11.28 (DM): now also JP4.2 (B); no longer TP2.1
- net at U11.29 (DP): now also JP5.2 (B)
- removed net ENC_B1: J1.2 (Pin_2), J5.4 (Pin_4)
- removed net ENC_C1: J5.5 (Pin_5), J9.2 (Pin_2)
- removed net VRAW: C18.1, J10.1, J7.1 (Pin_1), JP1.1 (A), JP2.2 (B), R43.2
- new net: JP7.2 (B), U6.A5 (CC1)
- new net: JP5.1 (A), U6.A6 (D+), U6.B6 (D+)
- new net: JP4.1 (A), U6.A7 (D-), U6.B7 (D-)
- new net: JP6.1 (A), U6.B5 (CC2)
- new net: C21.1, C22.1, FB1.2, U4.28 (VREF+), U4.29 (VDDA)
- new net Qi_CC1: JP7.1 (A)
- new net Qi_CC2: JP6.2 (B)
- new net V_QI_USB: JP1.1 (A), U6.A4 (VBUS), U6.A9 (VBUS), U6.B4 (VBUS), U6.B9 (VBUS)
- no-connect marks 20 -> 31
Other:
- note added: "long term: - max VIN is 18V from buck converter (upgrade?) - switch to smaller pkg drv SIG TODO: - better test probes - attach TEMP1 and TEMP2 to VOUT pins - fix wireless charger - change wireless chips to 0603 POWER TODO: - find power diode for D8 -pick new barrel jack? done: - improve SWD interface? (or is 4 pin jst good?) - change G432 to G474 - Boot button is actually rst (fix this) - add boo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"
- note removed: "long term: - max VIN is 18V from buck converter (upgrade?) - switch to smaller pkg drv SIG TODO: - power rate indicator LEDs - mode buttons with indicator - fix wireless charger - better test probes - current sns for wireless coil? - pick new SWD/I2C pins POWER TODO: - Bulk up RPP fet - do I need a power switch? - find power diode for D8 done: - improve SWD interface? (or is 4 pin jst good?) - ch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"
- moved on the sheet: C12, C14, C15, C16, C20, C21, C22, C23, C27, C28, C29, C30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
