File: I3ESC.kicad_sch (KiCad schematic)
At the start: 56 parts, among them J10 VIN_BARREL, J13 Conn_01x03, J5 Encoder1, J7 VIN_TERMINAL, J8 Encoder2, SW1 reset, SW2 boot-red, SW3 user1-white, U1 SY8113BADC, U11 Qwiic2, U3 SPX3819M5-L-3-3, U4 STM32G474RETx, U5 Qwiic1, U8 ABM3B-8.000MHZ

Commit message: update for summer 2026 production run
Parts:
- D42: LCSC C131795 -> C20612286
- D7: LCSC (none) -> C2286
- H1, H2, H3, H4: now not fitted
- J5: value Encoder1 -> Encoder
- J7: value VIN_TERMINAL -> Screw_Terminal_01x02; LCSC C8404 -> C557646
- J8: value Encoder2 -> Encoder
- SW1: value reset -> button; footprint AlfredoFootprints:Button_SKRKAEE020 -> AlfredoFootprints:button-3.6x6mm; LCSC C115357 -> C255802
- SW2: value boot-red -> button
- SW3: value user1-white -> button; LCSC C455236 -> C255802
- U11: value Qwiic2 -> Qwiic; LCSC C18077917 -> C51940129
- U5: value Qwiic1 -> Qwiic; LCSC C18077917 -> C51940129
Changed lines of the file:
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@@
 	)
 	(junction
-		(at 39.37 167.64)
-		(diameter 0)
-		(color 0 0 0 0)
-	)
-	(junction
 		(at 125.73 115.57)
 		(diameter 0)
@@
 	)
 	(junction
+		(at 39.37 167.64)
+		(diameter 0)
+		(color 0 0 0 0)
+	)
+	(junction
 		(at 127 168.91)
 		(diameter 0)
@@
 		(in_bom no)
 		(on_board yes)
-		(in_pos_files yes)
-		(dnp no)
+		(in_pos_files no)
+		(dnp yes)
 		(fields_autoplaced yes)
 		(property "Reference" "H2"
@@
 			)
 		)
-		(property "Value" "Qwiic1"
+		(property "Value" "Qwiic"
 			(at 207.01 72.39 0)
 			(show_name no)
@@
 			)
 		)
-		(property "Description" ""
+		(property "Description" "Qwiic1"
 			(at 205.74 78.74 0)
 			(hide yes)
@@
 			)
 		)
-		(property "LCSC" "C18077917"
+		(property "LCSC" "C51940129"
 			(at 205.74 78.74 0)
 			(hide yes)
@@
 			)
 		)
-		(property "Value" "Qwiic2"
+		(property "Value" "Qwiic"
 			(at 240.03 72.39 0)
 			(show_name no)
@@
 			)
 		)
-		(property "Description" ""
+		(property "Description" "Qwiic2"
 			(at 238.76 78.74 0)
 			(hide yes)
@@
 			)
 		)
-		(property "LCSC" "C18077917"
+		(property "LCSC" "C51940129"
 			(at 238.76 78.74 0)
 			(hide yes)
@@
 			)
 		)
-		(property "Value" "Encoder1"
+		(property "Value" "Encoder"
 			(at 251.714 100.076 0)
 			(show_name no)
@@
 			)
 		)
-		(property "Value" "user1-white"
-			(at 31.496 160.782 90)
+		(property "Value" "button"
+			(at 33.782 161.036 90)
 			(show_name no)
 			(do_not_autoplace no)
@@
 			)
 		)
-		(property "Description" ""
+		(property "Description" "User  Button"
 			(at 39.37 162.56 0)
 			(hide yes)
@@
 			)
 		)
-		(property "LCSC" "C455236"
+		(property "LCSC" "C255802"
 			(at 39.37 162.56 0)
 			(hide yes)
@@
 		(in_bom no)
 		(on_board yes)
-		(in_pos_files yes)
-		(dnp no)
+		(in_pos_files no)
+		(dnp yes)
 		(fields_autoplaced yes)
 		(property "Reference" "H1"
@@
 			)
 		)
-		(property "Value" "VIN_TERMINAL"
+		(property "Value" "Screw_Terminal_01x02"
 			(at 51.816 46.99 0)
 			(show_name no)
@@
 			)
 		)
-		(property "LCSC" "C8404 "
+		(property "LCSC" "C557646"
 			(at 48.26 41.91 0)
 			(hide yes)
@@
 			)
 		)
-		(property "LCSC" ""
+		(property "LCSC" "C2286 "
 			(at 185.42 144.78 0)
 			(hide yes)
@@
 		(in_bom no)
 		(on_board yes)
-		(in_pos_files yes)
-		(dnp no)
+		(in_pos_files no)
+		(dnp yes)
 		(fields_autoplaced yes)
 		(property "Reference" "H4"
@@
 			)
 		)
-		(property "LCSC" "C131795 "
+		(property "LCSC" "C20612286"
 			(at 223.52 144.78 0)
 			(hide yes)
@@
 			)
 		)
-		(property "Value" "reset"
+		(property "Value" "button"
 			(at 36.83 104.14 90)
 			(show_name no)
@@
 			)
 		)
-		(property "Footprint" "AlfredoFootprints:Button_SKRKAEE020"
+		(property "Footprint" "AlfredoFootprints:button-3.6x6mm"
 			(at 35.56 106.68 0)
 			(hide yes)
@@
 			)
 		)
-		(property "Datasheet" "https://lcsc.com/product-detail/Tactile-Switches_ALPSALPINE-ALPSALPINE-SKRKAEE020_C115357.html"
+		(property "Datasheet" "https://www.lcsc.com/product-detail/Tactile-Switches_HYP-Hongyuan-Precision-HYP-Hongyuan-Precision-1TS002E-2500-2501-CT_C255802.html"
 			(at 35.56 106.68 0)
 			(hide yes)
@@
 			)
 		)
-		(property "Description" ""
+		(property "Description" "Reset Button"
 			(at 40.64 106.68 0)
 			(hide yes)
@@
 			)
 		)
-		(property "LCSC" "C115357"
+		(property "LCSC" "C255802"
 			(at 40.64 106.68 0)
 			(hide yes)
@@
 			)
 		)
-		(property "Value" "Encoder2"
+		(property "Value" "Encoder"
 			(at 217.17 100.33 0)
 			(show_name no)
@@
 			)
 		)
-		(property "Value" "boot-red"
+		(property "Value" "button"
 			(at 32.258 127.762 90)
 			(show_name no)
@@
 			)
 		)
-		(property "Description" ""
+		(property "Description" "Boot Button"
 			(at 39.37 129.54 0)
 			(hide yes)
@@
 		(in_bom no)
 		(on_board yes)
-		(in_pos_files yes)
-		(dnp no)
+		(in_pos_files no)
+		(dnp yes)
 		(fields_autoplaced yes)
 		(property "Reference" "H3"

Commit message: fixed LCSC Numbers, order 9-10-26
Parts:
- D7: LCSC C2286 -> C2286
- D83: LCSC (none) -> C19171394
- D84: LCSC C2290 -> C2290
- J13: now left out of the parts list
- J5: LCSC C131342 -> C131342
- U11, U5: LCSC C51940129 -> C51940129
Other:
- note added: "Chips Used: STM32G474RET6 - C521608 - original STM32G473RCT6 - C529361 - value"
Changed lines of the file:
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@@
 		)
 	)
+	(text "Chips Used:\nSTM32G474RET6 - C521608 - original\nSTM32G473RCT6 - C529361 - value"
+		(exclude_from_sim no)
+		(at 17.018 66.802 0)
+		(effects
+			(font
+				(size 1.5 1.5)
+				(thickness 0.6)
+				(bold yes)
+			)
+			(justify left)
+		)
+	)
 	(text "POWER"
 		(exclude_from_sim no)
@@
 			)
 		)
-		(property "LCSC" "C51940129"
+		(property "LCSC" " C51940129"
 			(at 205.74 78.74 0)
 			(hide yes)
@@
 			)
 		)
-		(property "LCSC" "C51940129"
+		(property "LCSC" " C51940129"
 			(at 238.76 78.74 0)
 			(hide yes)
@@
 			)
 		)
-		(property "LCSC" " C131342"
+		(property "LCSC" "C131342"
 			(at 252.73 110.49 0)
 			(hide yes)
@@
 			)
 		)
-		(property "LCSC" " C2290"
+		(property "LCSC" "C2290"
 			(at 185.42 138.43 0)
 			(hide yes)
@@
 			)
 		)
-		(property "LCSC" "C2286 "
+		(property "LCSC" "C2286"
 			(at 185.42 144.78 0)
 			(hide yes)
@@
 			)
 		)
-		(property "LCSC" ""
+		(property "LCSC" "C19171394"
 			(at 185.42 132.08 0)
 			(hide yes)
@@
 		(body_style 1)
 		(exclude_from_sim no)
-		(in_bom yes)
+		(in_bom no)
 		(on_board yes)
 		(in_pos_files yes)
