File: I3ESC.kicad_pcb (KiCad board)
At the start: 4 copper layers, 45 x 17.4 mm, 97 parts, among them J1 PhaseOut, J2 PhaseOut, J3 PhaseOut, J30 CanOut, J4 GND, J40 Vin, J41 Gnd, J81 Conn_02x07_Counter_Clockwise, Q1 YJG150N03A, Q2 YJG150N03A, Q3 YJG150N03A, Q4 YJG150N03A, Q5 YJG150N03A, Q6 YJG150N03A, U2 FD8288T (DRV8300), U30 MCP2551-I-SN, U31 CPDT-12V, U4 INA185A1, U5 INA185A1, U50 SPX3819M5-L-3-3, U6 INA185A1, U60 SY8113BADC, U80 STM32F103CBTx, U81 ABM3B-8.000MHZ

Commit message: updated with g431 info
Parts:
- removed the C1 at (3.00, -7.60)
- removed the C10 at (2.00, -3.88)
- removed the C2 at (1.10, 0.00)
- removed the C3 at (3.00, 7.60)
- removed the C4 at (9.70, -0.30)
- removed the C40 at (4.40, 4.19)
- removed the C42 at (6.80, -3.30)
- removed the C5 at (9.70, 2.40)
- removed the C52 at (-12.5, 8.00)
- removed the C53 at (-14.3, 8.00)
- removed the C6 at (9.70, 4.80)
- removed the C60 at (-19.2, 7.25)
- removed the C61 at (-18.9, 2.20)
- removed the C62 at (-17.7, 6.40)
- removed the C63 at (-16.9, 2.20)
- removed the C7 at (16.1, -7.30)
- removed the C8 at (19.9, -1.70)
- removed the C80 at (-8.20, 0.00)
- removed the C81 at (-1.30, 4.60)
- removed the C82 at (-10.4, -4.60)
- removed the C83 at (-1.00, -4.30)
- removed the C84 at (-11.3, 2.10)
- removed the C88 at (-11.3, -1.45)
- removed the C89 at (-11.3, 0.30)
- removed the C9 at (19.7, 4.10)
- removed the D1 at (13.3, -7.50)
- removed the D2 at (12.8, -1.70)
- removed the D3 at (13.5, 4.10)
- removed the D4 at (9.80, -1.50)
- removed the D42 at (7.90, -4.70)
- removed the D5 at (10.0, 1.20)
- removed the D6 at (9.90, 3.65)
- removed the D83 at (3.55, 7.80)
- removed the D84 at (6.75, 7.80)
- removed the J1 at (23.0, -7.00)
- removed the J2 at (22.9, 0.00)
- removed the J3 at (23.0, 7.00)
- removed the J30 at (-18.2, -2.90)
- removed the J4 at (23.0, 3.50)
- removed the J40 at (-2.00, 7.00)
- removed the J81 at (-14.4, 0.00)
- removed the L60 at (-18.4, 2.16)
- removed the Q1 at (9.00, -5.70)
- removed the Q2 at (9.00, 0.10)
- removed the Q3 at (9.00, 5.90)
- removed the Q4 at (16.5, -5.70)
- removed the Q5 at (16.5, 0.10)
- removed the Q6 at (16.5, 5.90)
- removed the R1 at (16.4, -4.70)
- removed the R10 at (12.0, -5.70)
- removed the R11 at (12.0, 0.10)
- removed the R12 at (12.0, 5.90)
- removed the R13 at (11.2, -5.55)
- removed the R14 at (15.2, -1.80)
- removed the R15 at (11.2, 5.25)
- removed the R16 at (16.1, -8.15)
- removed the R17 at (19.1, -1.70)
- removed the R18 at (18.9, 4.10)
- removed the R19 at (12.0, -3.90)
- removed the R2 at (16.4, 1.10)
- removed the R21 at (12.0, 7.70)
- removed the R22 at (8.30, 6.05)
- removed the R23 at (2.10, 6.05)
- removed the R24 at (0.40, 4.40)
- removed the R3 at (16.4, 6.90)
- removed the R30 at (-7.00, 0.00)
- removed the R31 at (-6.05, 0.00)
- removed the R32 at (-11.3, -4.60)
- removed the R4 at (23.0, -3.35)
- removed the R40 at (3.80, -0.05)
- removed the R41 at (4.80, -0.05)
- removed the R42 at (6.80, -2.50)
- removed the R43 at (8.80, -3.30)
- removed the R60 at (-17.7, 7.30)
- removed the R61 at (-17.6, 8.15)
- removed the R7 at (23.0, -2.40)
- removed the R80 at (-5.10, 0.00)
- removed the R84 at (-9.80, 6.85)
- removed the R85 at (-9.80, 7.75)
- removed the TP80 at (-7.35, -6.25)
- removed the TP81 at (-6.55, -7.70)
- removed the TP83 at (-12.3, -7.70)
- removed the TP84 at (-8.10, -7.70)
- removed the U2 at (4.90, 2.10)
- removed the U30 at (-12.4, -6.10)
- removed the U31 at (-18.1, -6.90)
- removed the U4 at (18.3, -7.50)
- removed the U5 at (16.8, -1.80)
- removed the U50 at (-13.4, 5.60)
- removed the U6 at (16.8, 4.00)
- removed the U60 at (-17.9, 4.40)
- removed the U80 at (-5.60, 0.00)
- removed the U81 at (-10.8, 0.00)
- added ?: , , F.Cu at (255.8, 79.2)
- added ?: , , F.Cu at (182.7, 98.0)
- added ?: , , F.Cu at (222.9, 88.5)
- added C1: 4.7uF,50V, Capacitor_SMD:C_1206_3216Metric, F.Cu at (-46.8, -17.6)
- added C1: 10uF,25V, Capacitor_SMD:C_0805_2012Metric, F.Cu at (236.6, 83.0)
- added C1: 4.7uF,50V, Capacitor_SMD:C_1206_3216Metric, B.Cu at (139.5, 29.4)
- added C10: 10uF,50V, Capacitor_SMD:C_1206_3216Metric, F.Cu at (-73.1, -27.0)
- added C10: 10uF,50V, Capacitor_SMD:C_1206_3216Metric, F.Cu at (138.5, 33.1)
- added C10: 1uF?/24V?, Capacitor_SMD:C_0805_2012Metric, F.Cu at (204.3, 106.7)
- added C100: 0.8pF, Capacitor_SMD:C_0402_1005Metric, F.Cu at (-61.1, 30.9)
- added C101: 1.2pF, Capacitor_SMD:C_0402_1005Metric, F.Cu at (-58.2, 24.9)
- added C102: 1.2pF, Capacitor_SMD:C_0402_1005Metric, F.Cu at (-58.2, 26.9)
- added C103: 100pF, Capacitor_SMD:C_0402_1005Metric, F.Cu at (-58.2, 28.9)
- added C104: 0.5pF, Capacitor_SMD:C_0402_1005Metric, F.Cu at (-58.2, 30.9)
- added C11: 10nF, 6.3V, Capacitor_SMD:C_0402_1005Metric, F.Cu at (-57.7, -3.19)
- added C12: 22pF, Capacitor_SMD:C_0402_1005Metric, F.Cu at (-57.7, -1.23)
- added C13: 2.2uF, 6.3V, Capacitor_SMD:C_0402_1005Metric, F.Cu at (-57.7, 0.74)
- added C14: 2.2uF, 10V, Capacitor_SMD:C_0402_1005Metric, F.Cu at (-57.7, 2.71)
- added C15: 15pF, Capacitor_SMD:C_0402_1005Metric, F.Cu at (-83.3, -18.4)
- added C16: 15pF, Capacitor_SMD:C_0402_1005Metric, F.Cu at (-83.3, -16.4)
- added C17: 100nF, Capacitor_SMD:C_0402_1005Metric, F.Cu at (-83.3, -14.5)
- added C2: 4.7uF,50V, Capacitor_SMD:C_1206_3216Metric, F.Cu at (-46.8, -36.3)
- added C2: 10uF,25V, Capacitor_SMD:C_0805_2012Metric, F.Cu at (236.6, 93.0)
- added C2: 4.7uF,50V, Capacitor_SMD:C_1206_3216Metric, B.Cu at (137.6, 37.0)
- added C3: 4.7uF,50V, Capacitor_SMD:C_1206_3216Metric, F.Cu at (-84.0, 0.11)
- added C3: 10uF,25V, Capacitor_SMD:C_0805_2012Metric, F.Cu at (236.6, 103.0)
- added C3: 4.7uF,50V, Capacitor_SMD:C_1206_3216Metric, B.Cu at (139.5, 44.6)
- added C4: 1uF, Capacitor_SMD:C_0402_1005Metric, F.Cu at (146.2, 36.7)
- added C4: 470nF?/16V?, Capacitor_SMD:C_0603_1608Metric, F.Cu at (216.0, 101.6)
- added C4: 1uF, Capacitor_SMD:C_0402_1005Metric, F.Cu at (-83.3, -24.3)
- added C40: 330uF, AlfredoFootprints:TGD_lowESR_cap, F.Cu at (240.4, 76.0)
- added C40: 330uF, AlfredoFootprints:Cap_THT_LowESR_330uF, B.Cu at (140.9, 41.2)
- added C42: 100nF, Capacitor_SMD:C_0603_1608Metric, F.Cu at (250.6, 73.7)
- added C42: 100nF, Capacitor_SMD:C_0402_1005Metric, F.Cu at (-80.4, -24.3)
- added C42: 100nF, Capacitor_SMD:C_0402_1005Metric, F.Cu at (143.3, 33.7)
- added C5: 1uF, Capacitor_SMD:C_0402_1005Metric, F.Cu at (-83.3, -22.3)
- added C5: 470nF?/16V?, Capacitor_SMD:C_0603_1608Metric, F.Cu at (216.0, 104.6)
- added C5: 1uF, Capacitor_SMD:C_0402_1005Metric, F.Cu at (146.2, 39.4)
- added C50: 10uF, Capacitor_SMD:C_0603_1608Metric, F.Cu at (197.7, 97.3)
- added C51: 100nF, Capacitor_SMD:C_0603_1608Metric, F.Cu at (192.5, 97.3)
- added C52: 22pF, Capacitor_SMD:C_0603_1608Metric, F.Cu at (195.1, 101.3)
- added C52: 10nF, 6.3V, Capacitor_SMD:C_0402_1005Metric, B.Cu at (124.0, 45.0)
- added C53: 22uF, Capacitor_SMD:C_0603_1608Metric, F.Cu at (192.5, 100.5)
- added C53: 2.2uF, 6.3V, Capacitor_SMD:C_0402_1005Metric, B.Cu at (122.2, 45.0)
- added C6: 470nF?/16V?, Capacitor_SMD:C_0603_1608Metric, F.Cu at (216.0, 107.6)
- added C6: 1uF, Capacitor_SMD:C_0402_1005Metric, F.Cu at (-83.3, -20.4)
- added C6: 1uF, Capacitor_SMD:C_0402_1005Metric, F.Cu at (146.2, 41.8)
- added C60: 10pF, Capacitor_SMD:C_0402_1005Metric, F.Cu at (-66.8, 24.9)
- added C60: 10uF, Capacitor_SMD:C_0603_1608Metric, F.Cu at (197.7, 105.1)
- added C60: 2.2uF, 50V, Capacitor_SMD:C_0603_1608Metric, B.Cu at (117.3, 44.2)
- added C61: 10pF, Capacitor_SMD:C_0402_1005Metric, F.Cu at (-66.8, 26.9)
- added C61: 100nF, Capacitor_SMD:C_0603_1608Metric, F.Cu at (192.5, 105.1)
- added C61: 100nF, Capacitor_SMD:C_0402_1005Metric, B.Cu at (117.6, 39.2)
- added C62: 2.2uF, Capacitor_SMD:C_0402_1005Metric, F.Cu at (-66.8, 28.9)
- added C62: 22pF, Capacitor_SMD:C_0603_1608Metric, F.Cu at (195.1, 109.1)
- added C62: 22pF, Capacitor_SMD:C_0402_1005Metric, B.Cu at (118.8, 43.4)
- added C63: 100nF, Capacitor_SMD:C_0402_1005Metric, F.Cu at (-66.8, 30.9)
- added C63: 22uF, Capacitor_SMD:C_0603_1608Metric, F.Cu at (192.5, 108.3)
- added C63: 22uF, 10V, Capacitor_SMD:C_0402_1005Metric, B.Cu at (119.6, 39.2)
- added C64: 2.2uF, Capacitor_SMD:C_0402_1005Metric, F.Cu at (-64.0, 24.9)
- added C65: 2.2uF, Capacitor_SMD:C_0402_1005Metric, F.Cu at (-64.0, 26.9)
- added C7: 4.7nF, Capacitor_SMD:C_0402_1005Metric, F.Cu at (152.7, 29.7)
- added C7: 4.7nF, Capacitor_SMD:C_0603_1608Metric, F.Cu at (246.7, 84.1)
- added C7: 4.7nF, Capacitor_SMD:C_0402_1005Metric, F.Cu at (-55.7, -13.5)
- added C70: 2.2uF, Capacitor_SMD:C_0402_1005Metric, F.Cu at (-64.0, 28.9)
- added C71: 10nF, Capacitor_SMD:C_0402_1005Metric, F.Cu at (-64.0, 30.9)
- added C72: 100nF, Capacitor_SMD:C_0402_1005Metric, F.Cu at (-61.1, 24.9)
- added C73: 100nF, Capacitor_SMD:C_0402_1005Metric, F.Cu at (-61.1, 26.9)
- added C74: 10nF, Capacitor_SMD:C_0402_1005Metric, F.Cu at (-61.1, 28.9)
- added C8: 4.7nF, Capacitor_SMD:C_0402_1005Metric, F.Cu at (-55.7, -32.2)
- added C8: 4.7nF, Capacitor_SMD:C_0603_1608Metric, F.Cu at (246.7, 94.1)
- added C8: 4.7nF, Capacitor_SMD:C_0402_1005Metric, F.Cu at (156.4, 35.3)
- added C80: 100nF, Capacitor_SMD:C_0603_1608Metric, F.Cu at (176.9, 80.5)
- added C80: 100nF, Capacitor_SMD:C_0402_1005Metric, B.Cu at (128.3, 37.0)
- added C800: 2.2uF, 50V, Capacitor_SMD:C_0603_1608Metric, F.Cu at (-66.8, 19.9)
- added C81: 2.2uF, 10V, Capacitor_SMD:C_0402_1005Metric, F.Cu at (-80.4, -22.3)
- added C81: 2.2uF, Capacitor_SMD:C_0603_1608Metric, F.Cu at (177.3, 74.7)
- added C81: 2.2uF, 10V, Capacitor_SMD:C_0402_1005Metric, F.Cu at (135.2, 41.6)
- added C82: 2.2uF, Capacitor_SMD:C_0603_1608Metric, F.Cu at (187.5, 86.0)
- added C82: 2.2uF, 10V, Capacitor_SMD:C_0402_1005Metric, F.Cu at (126.1, 32.4)
- added C82: 2.2uF, 10V, Capacitor_SMD:C_0402_1005Metric, F.Cu at (-80.4, -20.4)
- added C83: 2.2uF, 10V, Capacitor_SMD:C_0402_1005Metric, F.Cu at (-80.4, -18.4)
- added C83: 2.2uF, Capacitor_SMD:C_0603_1608Metric, F.Cu at (190.5, 76.2)
- added C83: 2.2uF, 10V, Capacitor_SMD:C_0402_1005Metric, F.Cu at (135.5, 32.7)
- added C84: 2.2uF, 10V, Capacitor_SMD:C_0402_1005Metric, F.Cu at (125.2, 39.1)
- added C84: 2.2uF, Capacitor_SMD:C_0603_1608Metric, F.Cu at (181.1, 73.5)
- added C84: 2.2uF, 10V, Capacitor_SMD:C_0402_1005Metric, F.Cu at (-80.4, -16.4)
- added C85: 2.2uF, Capacitor_SMD:C_0603_1608Metric, F.Cu at (177.6, 82.9)
- added C88: 15pF, Capacitor_SMD:C_0402_1005Metric, F.Cu at (125.2, 35.5)
- added C88: 15pF, Capacitor_SMD:C_0603_1608Metric, F.Cu at (174.3, 74.7)
- added C89: 15pF, Capacitor_SMD:C_0402_1005Metric, F.Cu at (125.2, 37.3)
- added C89: 15pF, Capacitor_SMD:C_0603_1608Metric, F.Cu at (173.7, 80.5)
- added C9: 4.7nF, Capacitor_SMD:C_0603_1608Metric, F.Cu at (246.7, 104.1)
- added C9: 4.7nF, Capacitor_SMD:C_0402_1005Metric, F.Cu at (-93.0, 4.15)
- added C9: 4.7nF, Capacitor_SMD:C_0402_1005Metric, F.Cu at (156.2, 41.1)
- added C900: 100nF, Capacitor_SMD:C_0402_1005Metric, F.Cu at (-57.7, 4.68)
- added D1: ZMM3V3, Diode_SMD:D_MiniMELF, F.Cu at (241.1, 82.9)
- added D1: Z3V3, Diode_SMD:D_SOD-323_HandSoldering, F.Cu at (149.8, 29.5)
- added D1: Z3V3, Diode_SMD:D_SOD-323_HandSoldering, F.Cu at (-47.0, -14.4)
- added D2: Z3V3, Diode_SMD:D_SOD-323_HandSoldering, F.Cu at (149.3, 35.3)
- added D2: Z3V3, Diode_SMD:D_SOD-323_HandSoldering, F.Cu at (-47.0, -33.1)
- added D2: ZMM3V3, Diode_SMD:D_MiniMELF, F.Cu at (241.1, 92.9)
- added D3: Z3V3, Diode_SMD:D_SOD-323_HandSoldering, F.Cu at (-84.3, 3.26)
- added D3: Z3V3, Diode_SMD:D_SOD-323_HandSoldering, F.Cu at (150.0, 41.1)
- added D3: ZMM3V3, Diode_SMD:D_MiniMELF, F.Cu at (241.1, 103.0)
- added D4: SDM20U40-7, Diode_SMD:D_SOD-523, F.Cu at (-65.3, -19.2)
- added D4: SDM20U40-7, Diode_SMD:D_SOD-523, F.Cu at (146.3, 35.5)
- added D4: CRH01, Diode_SMD:D_SOD-123F, F.Cu at (221.1, 100.8)
- added D40: B5819W, Diode_SMD:D_SOD-123, F.Cu at (187.2, 107.4)
- added D41: B5819W, Diode_SMD:D_SOD-123, F.Cu at (201.5, 99.6)
- added D42: Z3V3, Diode_SMD:D_SOD-323_HandSoldering, F.Cu at (144.4, 32.3)
- added D42: ZMM3V3, Diode_SMD:D_MiniMELF, F.Cu at (246.5, 74.8)
- added D42: Z3V3, Diode_SMD:D_SOD-323_HandSoldering, F.Cu at (-95.6, -16.1)
- added D5: SDM20U40-7, Diode_SMD:D_SOD-523, F.Cu at (-65.3, -16.8)
- added D5: SDM20U40-7, Diode_SMD:D_SOD-523, F.Cu at (146.5, 38.2)
- added D5: CRH01, Diode_SMD:D_SOD-123F, F.Cu at (221.1, 103.8)
- added D6: SDM20U40-7, Diode_SMD:D_SOD-523, F.Cu at (-65.3, -14.3)
- added D6: CRH01, Diode_SMD:D_SOD-123F, F.Cu at (221.1, 106.8)
- added D6: SDM20U40-7, Diode_SMD:D_SOD-523, F.Cu at (146.4, 40.6)
- added D60: LED_yellow, LED_SMD:LED_0603_1608Metric, F.Cu at (-66.2, 40.4)
- added D7: Z5V6, AlfredoFootprints:D_SOD-323, F.Cu at (-65.5, -37.5)
- added D70: Z3V3, Diode_SMD:D_MiniMELF, F.Cu at (208.0, 88.8)
- added D71: Z3V3, Diode_SMD:D_MiniMELF, F.Cu at (208.0, 91.2)
- added D72: Z3V3, Diode_SMD:D_MiniMELF, F.Cu at (208.1, 77.0)
- added D73: Z3V3, Diode_SMD:D_MiniMELF, F.Cu at (208.1, 74.6)
- added D74: Z3V3, Diode_SMD:D_MiniMELF, F.Cu at (208.1, 84.2)
- added D75: Z3V3, Diode_SMD:D_MiniMELF, F.Cu at (208.1, 79.4)
- added D76: Z3V3, Diode_SMD:D_MiniMELF, F.Cu at (208.1, 81.8)
- added D77: Z3V3, Diode_SMD:D_MiniMELF, F.Cu at (208.1, 72.2)
- added D80: LED_Dual_AKA, LED_THT:LED_D3.0mm-3, F.Cu at (168.9, 96.6)
- added D81: LED_Dual_AKA, LED_THT:LED_D3.0mm-3, F.Cu at (161.9, 96.5)
- added D83: LED_Red, LED_SMD:LED_0805_2012Metric, F.Cu at (-65.3, -33.7)
- added D83: LED_Red, LED_SMD:LED_0805_2012Metric, F.Cu at (140.1, 44.8)
- added D84: LED_Green, LED_SMD:LED_0805_2012Metric, F.Cu at (-65.3, -30.7)
- added D84: LED_Green, LED_SMD:LED_0805_2012Metric, F.Cu at (143.2, 44.8)
- added G***: LOGO, AlfredoFootprints:Alfredo_logo_small, B.Cu at (252.5, 78.8)
- added H1: MountingHole, AlfredoFootprints:TGD_MountingHole, F.Cu at (-94.5, -43.0)
- added H2: MountingHole, AlfredoFootprints:TGD_MountingHole, F.Cu at (-94.5, -35.7)
- added H3: MountingHole, AlfredoFootprints:TGD_MountingHole, F.Cu at (-94.5, -28.5)
- added H4: MountingHole, AlfredoFootprints:TGD_MountingHole, F.Cu at (-94.5, -21.2)
- added J1: PhaseOut, AlfredoFootprints:TGD_ESC_PwrPad, F.Cu at (254.7, 87.7)
- added J1: PhaseOut, AlfredoFootprints:GE_PwrPad1, F.Cu at (159.5, 30.0)
- added J1: PhaseOut, AlfredoFootprints:GE_PwrPad1, F.Cu at (-47.0, -21.1)
- added J10: Conn_01x06, Connector_PinSocket_2.54mm:PinSocket_1x06_P2.54mm_Vertical, F.Cu at (192.8, 91.4)
- added J2: PhaseOut, AlfredoFootprints:GE_PwrPad1, F.Cu at (159.4, 37.0)
- added J2: PhaseOut, AlfredoFootprints:TGD_ESC_PwrPad, F.Cu at (254.7, 97.7)
- added J2: PhaseOut, AlfredoFootprints:GE_PwrPad1, F.Cu at (-47.0, -39.8)
- added J3: PhaseOut, AlfredoFootprints:TGD_ESC_PwrPad, F.Cu at (254.6, 107.7)
- added J3: PhaseOut, AlfredoFootprints:GE_PwrPad1, F.Cu at (-84.2, -3.44)
- added J3: PhaseOut, AlfredoFootprints:GE_PwrPad1, F.Cu at (159.5, 44.0)
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Connections:
- R20 pad 1: Net-(Q2-Pad4) -> (no net)
- R20 pad 2: /GE-Fets-B/GHx -> (no net)
Routing:
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- added copper zone on B.Cu, net (none)
- added copper zone on F.Cu, net (none)
- added copper zone on In2.Cu, net +3V3
- added copper zone on B.Cu, net /IE-Fets-A/SHx
- added copper zone on F.Cu, net /IE-Fets-A/SHx
- added copper zone on B.Cu, net /IE-Fets-B/SHx
- added copper zone on F.Cu, net /IE-Fets-B/SHx
- added copper zone on B.Cu, net /IE-Fets-C/SHx
- added copper zone on F.Cu, net /IE-Fets-C/SHx
- added copper zone on F.Cu, net Net-(J1-Pin_1)
- added copper zone on F.Cu, net Net-(J2-Pin_1)
- added copper zone on F.Cu, net Net-(J3-Pin_1)
- removed copper zone on B.Cu, net /GE-Fets-A/SHx
- removed copper zone on F.Cu, net /GE-Fets-A/SHx
- removed copper zone on B.Cu, net /GE-Fets-B/SHx
- removed copper zone on F.Cu, net /GE-Fets-B/SHx
- removed copper zone on B.Cu, net /GE-Fets-C/SHx
- removed copper zone on F.Cu, net /GE-Fets-C/SHx
- removed copper zone on F.Cu, net Net-(J1-Pad1)
- removed copper zone on F.Cu, net Net-(J2-Pad1)
- removed copper zone on F.Cu, net Net-(J3-Pad1)
Other:
- board size 45 x 17.4 mm -> 141 x 82.4 mm
- board text added: "3V3"
- board text added: "5V"
- board text added: "CanH"
- board text added: "CanL"
- board text added: "GoldESC V1 © Alfredo Systems 2022"
- board text added: "HA"
- board text added: "HB"
- board text added: "HC"
- board text added: "LA"
- board text added: "LB"
- board text added: "LC"
- board text added: "SWCLK"
- board text added: "SWDIO"

Commit message: push before removing bldc1 external opAmps
Parts:
- removed ? (x3): , 
- removed the C1 at (-46.8, -17.6)
- removed the C1 at (236.6, 83.0)
- removed the C1 at (139.5, 29.4)
- removed the C10 at (-73.1, -27.0)
- removed the C10 at (138.5, 33.1)
- removed the C10 at (204.3, 106.7)
- removed C100: 0.8pF, Capacitor_SMD:C_0402_1005Metric
- removed C101, C102: 1.2pF, Capacitor_SMD:C_0402_1005Metric
- removed C103: 100pF, Capacitor_SMD:C_0402_1005Metric
- removed C104: 0.5pF, Capacitor_SMD:C_0402_1005Metric
- removed the C2 at (-46.8, -36.3)
- removed the C2 at (236.6, 93.0)
- removed the C2 at (137.6, 37.0)
- removed the C3 at (-84.0, 0.11)
- removed the C3 at (236.6, 103.0)
- removed the C3 at (139.5, 44.6)
- removed the C4 at (146.2, 36.7)
- removed the C4 at (216.0, 101.6)
- removed the C4 at (-83.3, -24.3)
- removed the C40 at (240.4, 76.0)
- removed the C40 at (140.9, 41.2)
- removed the C42 at (250.6, 73.7)
- removed the C42 at (-80.4, -24.3)
- removed the C42 at (143.3, 33.7)
- removed the C5 at (-83.3, -22.3)
- removed the C5 at (216.0, 104.6)
- removed the C5 at (146.2, 39.4)
- removed C50, C60: 10uF, Capacitor_SMD:C_0603_1608Metric
- removed C51, C61, C80: 100nF, Capacitor_SMD:C_0603_1608Metric
- removed C52, C62: 22pF, Capacitor_SMD:C_0603_1608Metric
- removed C52: 10nF, 6.3V, Capacitor_SMD:C_0402_1005Metric
- removed C53, C63: 22uF, Capacitor_SMD:C_0603_1608Metric
- removed C53: 2.2uF, 6.3V, Capacitor_SMD:C_0402_1005Metric
- removed the C6 at (216.0, 107.6)
- removed the C6 at (-83.3, -20.4)
- removed the C6 at (146.2, 41.8)
- removed C60, C61: 10pF, Capacitor_SMD:C_0402_1005Metric
- removed C60: 2.2uF, 50V, Capacitor_SMD:C_0603_1608Metric
- removed C61, C63, C72, C73, C80: 100nF, Capacitor_SMD:C_0402_1005Metric
- removed C62, C64, C65, C70: 2.2uF, Capacitor_SMD:C_0402_1005Metric
- removed C62: 22pF, Capacitor_SMD:C_0402_1005Metric
- removed C63: 22uF, 10V, Capacitor_SMD:C_0402_1005Metric
- removed the C7 at (152.7, 29.7)
- removed the C7 at (246.7, 84.1)
- removed the C7 at (-55.7, -13.5)
- removed C71, C74: 10nF, Capacitor_SMD:C_0402_1005Metric
- removed the C8 at (-55.7, -32.2)
- removed the C8 at (246.7, 94.1)
- removed the C8 at (156.4, 35.3)
- removed C81 (x2), C82 (x2), C83 (x2), C84 (x2): 2.2uF, 10V, Capacitor_SMD:C_0402_1005Metric
- removed C81, C82, C83, C84, C85: 2.2uF, Capacitor_SMD:C_0603_1608Metric
- removed C88, C89: 15pF, Capacitor_SMD:C_0402_1005Metric
- removed C88, C89: 15pF, Capacitor_SMD:C_0603_1608Metric
- removed the C9 at (246.7, 104.1)
- removed the C9 at (-93.0, 4.15)
- removed the C9 at (156.2, 41.1)
- removed the D1 at (241.1, 82.9)
- removed the D1 at (149.8, 29.5)
- removed the D1 at (-47.0, -14.4)
- removed the D2 at (149.3, 35.3)
- removed the D2 at (-47.0, -33.1)
- removed the D2 at (241.1, 92.9)
- removed the D3 at (-84.3, 3.26)
- removed the D3 at (150.0, 41.1)
- removed the D3 at (241.1, 103.0)
- removed the D4 at (-65.3, -19.2)
- removed the D4 at (146.3, 35.5)
- removed the D4 at (221.1, 100.8)
- removed D40, D41: B5819W, Diode_SMD:D_SOD-123
- removed the D42 at (144.4, 32.3)
- removed the D42 at (246.5, 74.8)
- removed the D42 at (-95.6, -16.1)
- removed the D5 at (-65.3, -16.8)
- removed the D5 at (146.5, 38.2)
- removed the D5 at (221.1, 103.8)
- removed the D6 at (-65.3, -14.3)
- removed the D6 at (221.1, 106.8)
- removed the D6 at (146.4, 40.6)
- removed D60: LED_yellow, LED_SMD:LED_0603_1608Metric
- removed D70, D71, D72, D73, D74, D75, D76, D77: Z3V3, Diode_SMD:D_MiniMELF
- removed D80, D81: LED_Dual_AKA, LED_THT:LED_D3.0mm-3
- removed the D83 at (-65.3, -33.7)
- removed the D83 at (140.1, 44.8)
- removed the D84 at (-65.3, -30.7)
- removed the D84 at (143.2, 44.8)
- removed G***: LOGO, AlfredoFootprints:Alfredo_logo_small
- removed the J1 at (254.7, 87.7)
- removed the J1 at (159.5, 30.0)
- removed the J1 at (-47.0, -21.1)
- removed the J2 at (159.4, 37.0)
- removed the J2 at (254.7, 97.7)
- removed the J2 at (-47.0, -39.8)
- removed the J3 at (254.6, 107.7)
- removed the J3 at (-84.2, -3.44)
- removed the J3 at (159.5, 44.0)
- removed J30 (x2): CanOut, AlfredoFootprints:GE_SigPad_1x02
- removed J30: CanOut, AlfredoFootprints:TGD_ESC_SigPads
- removed the J4 at (159.5, 40.5)
- removed the J4 at (-88.3, -15.0)
- removed J40: Vin, AlfredoFootprints:GE_PwrPad1
- removed J40: Supply, TerminalBlock:TerminalBlock_bornier-2_P5.08mm
- removed J41: Gnd, AlfredoFootprints:GE_PwrPad1
- removed J60: Conn_Coaxial, Connector_Coaxial:U.FL_Hirose_U.FL-R-SMT-1_Vertical
- removed J61: RFANT3216120A5T, Capacitor_SMD:C_1206_3216Metric
- removed J81 (x2): Conn_02x07_Counter_Clockwise, AlfredoFootprints:Connector_2x05_P1.27mm_IDC
- removed J81: Conn_02x07_Counter_Clockwise, Connector_IDC:IDC-Header_2x07_P2.54mm_Vertical
- removed J82: Conn_01x06, Connector_PinSocket_2.54mm:PinSocket_1x06_P2.54mm_Vertical
- removed L101: 3nH, Inductor_SMD:L_0402_1005Metric
- removed L102: 2.5nH, Inductor_SMD:L_0402_1005Metric
- removed L30: KCZ1210, AlfredoFootprints:KCZ1210
- removed L50, L60 (x2): 4.7uH, Inductor_SMD:L_1210_3225Metric
- removed the Q1 at (238.6, 86.9)
- removed the Q1 at (-56.9, -24.5)
- removed the Q1 at (145.5, 31.3)
- removed the Q2 at (-56.9, -43.2)
- removed the Q2 at (238.6, 96.9)
- removed the Q2 at (145.5, 37.1)
- removed the Q3 at (-94.1, -6.79)
- removed the Q3 at (238.6, 107.0)
- removed the Q3 at (145.5, 42.9)
- removed the Q4 at (-56.9, -17.8)
- removed the Q4 at (153.0, 31.3)
- removed the Q4 at (238.6, 86.9)
- removed the Q5 at (-56.9, -36.5)
- removed the Q5 at (153.0, 37.1)
- removed the Q5 at (238.6, 96.9)
- removed the Q6 at (-94.1, -0.10)
- removed the Q6 at (153.0, 42.9)
- removed the Q6 at (238.6, 107.0)
- removed the R1 at (152.9, 32.3)
- removed the R1 at (248.1, 87.7)
- removed the R1 at (-48.2, -25.4)
- removed the R10 at (148.5, 31.3)
- removed the R10 at (-51.0, -22.0)
- removed the R10 at (244.3, 84.8)
- removed the R11 at (148.5, 37.1)
- removed the R11 at (-51.0, -40.7)
- removed the R11 at (244.3, 94.8)
- removed the R12 at (-88.3, -4.32)
- removed the R12 at (148.5, 42.9)
- removed the R12 at (244.3, 104.8)
- removed the R13 at (245.0, 82.5)
- removed the R13 at (-51.0, -20.0)
- removed the R13 at (147.7, 31.4)
- removed the R14 at (-51.0, -38.7)
- removed the R14 at (245.0, 92.5)
- removed the R14 at (151.7, 35.2)
- removed the R15 at (245.0, 102.5)
- removed the R15 at (-88.3, -2.33)
- removed the R15 at (147.7, 42.2)
- removed the R16 at (-51.0, -18.0)
- removed the R16 at (248.9, 82.6)
- removed the R16 at (152.7, 28.9)
- removed the R17 at (-51.0, -36.7)
- removed the R17 at (248.9, 92.6)
- removed the R17 at (155.6, 35.3)
- removed the R18 at (248.9, 102.6)
- removed the R18 at (-88.3, -0.34)
- removed the R18 at (155.3, 41.1)
- removed the R19 at (229.9, 86.8)
- removed the R19 at (-51.0, -16.0)
- removed the R19 at (148.5, 33.1)
- removed the R2 at (248.1, 97.7)
- removed the R2 at (-48.2, -44.2)
- removed the R2 at (152.9, 38.1)
- removed the R21 at (144.8, 43.0)
- removed the R21 at (229.9, 106.8)
- removed the R21 at (-51.0, -14.0)
- removed the R22 at (-51.0, -34.7)
- removed the R22 at (148.5, 38.9)
- removed the R22 at (229.9, 85.0)
- removed the R23 at (138.6, 43.0)
- removed the R23 at (229.9, 95.0)
- removed the R23 at (-51.0, -32.8)
- removed the R24 at (148.5, 44.7)
- removed the R24 at (-88.3, 1.65)
- removed the R24 at (229.9, 105.0)
- removed the R25 at (-88.3, 3.64)
- removed the R25 at (136.9, 41.4)
- removed the R3 at (-85.4, -7.76)
- removed the R3 at (152.9, 43.9)
- removed the R3 at (248.1, 107.8)
- removed the R30 at (-80.3, -34.3)
- removed the R30 at (181.8, 102.5)
- removed the R30 at (129.5, 37.0)
- removed the R31 at (-80.3, -32.3)
- removed the R31 at (181.8, 104.1)
- removed the R31 at (130.4, 37.0)
- removed R32 (x2): 51K, Resistor_SMD:R_0402_1005Metric
- removed R32: 50K?, Resistor_THT:R_Axial_DIN0207_L6.3mm_D2.5mm_P10.16mm_Horizontal
- removed the R4 at (251.1, 83.3)
- removed the R4 at (-83.2, -34.3)
- removed the R4 at (159.5, 33.6)
- removed the R40 at (-80.3, -28.3)
- removed the R40 at (235.8, 90.4)
- removed the R40 at (140.3, 37.0)
- removed the R41 at (-80.3, -26.3)
- removed the R41 at (238.8, 90.4)
- removed the R41 at (141.3, 37.0)
- removed the R42 at (248.8, 73.7)
- removed the R42 at (-77.4, -34.3)
- removed the R42 at (143.3, 34.5)
- removed the R43 at (248.8, 76.7)
- removed the R43 at (-77.4, -32.3)
- removed the R43 at (145.3, 33.7)
- removed the R5 at (-83.2, -32.3)
- removed the R5 at (251.1, 93.3)
- removed the R6 at (251.1, 103.3)
- removed the R6 at (-83.2, -30.3)
- removed the R60 at (199.5, 108.3)
- removed the R60 at (-72.6, 28.9)
- removed the R60 at (118.8, 44.3)
- removed the R61 at (197.7, 108.3)
- removed the R61 at (118.8, 45.1)
- removed R66, R67: 1K, Resistor_SMD:R_0402_1005Metric
- removed R68: 330R, Resistor_SMD:R_0402_1005Metric
- removed the R7 at (252.6, 83.3)
- removed the R7 at (159.5, 34.6)
- removed the R7 at (-83.2, -28.3)
- removed R70, R71, R72, R73, R74, R75, R76, R77: 2K2, Resistor_SMD:R_0603_1608Metric
- removed the R8 at (252.6, 93.3)
- removed the R8 at (-83.2, -26.3)
- removed R80: 10K, Resistor_SMD:R_0603_1608Metric
- removed R80: 10K, Resistor_SMD:R_0402_1005Metric
- removed R81, R82: 22R, Resistor_SMD:R_0603_1608Metric
- removed R83, R84, R85, R86: 200R, Resistor_SMD:R_0603_1608Metric
- removed R84 (x2), R85 (x2): 200R, Resistor_SMD:R_0402_1005Metric
- removed the TP1 at (242.9, 81.0)
- removed the TP1 at (-68.5, -19.1)
- removed TP11, TP12, TP13, TP14, TP15, TP30, TP31, TP32, TP33, TP40, TP41, TP50, TP80 (x2), TP81 (x2), TP82: TestPoint, AlfredoFootprints:GE_TestPoint_Loop
- removed the TP83 at (124.2, 29.3)
- removed the TP83 at (-68.5, -16.3)
- removed the TP84 at (128.4, 29.3)
- removed the TP84 at (-68.5, -13.6)
- removed the U2 at (141.4, 39.1)
- removed the U2 at (-74.2, -21.3)
- removed the U2 at (209.7, 105.0)
- removed U30 (x3): MCP2551-I-SN, Package_SO:SOIC-8_3.9x4.9mm_P1.27mm
- removed U31 (x3): CPDT-12V, Package_TO_SOT_SMD:SOT-23
- removed the U4 at (154.8, 29.5)
- removed the U4 at (-59.0, -12.8)
- removed the U4 at (248.9, 84.5)
- removed the U5 at (248.9, 94.5)
- removed the U5 at (-59.0, -31.5)
- removed the U5 at (153.3, 35.2)
- removed U50, U60 (x2): SY8113BADC, Package_TO_SOT_SMD:TSOT-23-6
- removed U50: SPX3819M5-L-3-3, Package_TO_SOT_SMD:SOT-23-5
- removed the U6 at (153.3, 41.0)
- removed the U6 at (248.9, 104.5)
- removed the U6 at (-96.3, 4.91)
- removed U60: ESP8285H16, Package_DFN_QFN:QFN-32-1EP_5x5mm_P0.5mm_EP3.7x3.7mm
- removed U61: Crystal_ESP8285, Crystal:Crystal_SMD_2016-4Pin_2.0x1.6mm
- removed U70: SX1280, Package_DFN_QFN:QFN-24-1EP_4x4mm_P0.5mm_EP2.65x2.65mm
- removed U71: Crystal_SX1280, Crystal:Crystal_SMD_2016-4Pin_2.0x1.6mm
- removed U80 (x2): STM32F103CBTx, Package_QFP:LQFP-48_7x7mm_P0.5mm
- removed U80: STM32F103C8Tx, Package_QFP:LQFP-48_7x7mm_P0.5mm
- removed U81: Crystal_GND3, Crystal:Crystal_SMD_5032-4Pin_5.0x3.2mm
- removed U81: ABM3B-8.000MHZ, Crystal:Crystal_SMD_5032-4Pin_5.0x3.2mm
- added C1: 4.7uF,50V, Capacitor_SMD:C_1206_3216Metric, F.Cu at (-47.4, -87.7)
- added C10: 10uF,50V, Capacitor_SMD:C_1206_3216Metric, F.Cu at (-53.6, -118.6)
- added C18: 220uF, Capacitor_SMD:CP_Elec_6.3x7.7, F.Cu at (21.0, -46.0)
- added C19: 220uF, Capacitor_SMD:CP_Elec_6.3x7.7, F.Cu at (21.0, -37.9)
- added C2: 4.7uF,50V, Capacitor_SMD:C_1206_3216Metric, F.Cu at (-47.4, -84.3)
- added C20: 2.2uF, 10V, Capacitor_SMD:C_0402_1005Metric, F.Cu at (-139.5, 31.5)
- added C21: 2.2uF, 10V, Capacitor_SMD:C_0402_1005Metric, F.Cu at (-139.5, 33.5)
- added C22: 2.2uF, 10V, Capacitor_SMD:C_0402_1005Metric, F.Cu at (-139.5, 35.5)
- added C23: 2.2uF, 10V, Capacitor_SMD:C_0402_1005Metric, F.Cu at (-139.5, 37.4)
- added C24: 390pF, Capacitor_SMD:C_0402_1005Metric, F.Cu at (-2.36, -45.5)
- added C25: 390pF, Capacitor_SMD:C_0402_1005Metric, F.Cu at (-2.36, -43.5)
- added C26: 100nF, 50V, Capacitor_SMD:C_0402_1005Metric, F.Cu at (-2.36, -41.6)
- added C27: 100nF, Capacitor_SMD:C_0402_1005Metric, F.Cu at (72.3, 25.0)
- added C28: 100nF, Capacitor_SMD:C_0402_1005Metric, F.Cu at (72.3, 27.0)
- added C29: 250nF, Capacitor_THT:C_Rect_L9.0mm_W4.0mm_P7.50mm_MKT, F.Cu at (46.2, 5.00)
- added C3: 4.7uF,50V, Capacitor_SMD:C_1206_3216Metric, F.Cu at (-47.4, -81.0)
- added C30: 15nF, Capacitor_SMD:C_0402_1005Metric, F.Cu at (72.3, 28.9)
- added C31: 15nF, Capacitor_SMD:C_0402_1005Metric, F.Cu at (72.3, 30.9)
- added C32: 100nF, Capacitor_SMD:C_0402_1005Metric, F.Cu at (72.3, 32.9)
- added C33: 10uF,50V, Capacitor_SMD:C_1206_3216Metric, F.Cu at (76.5, 25.7)
- added C34: 10uF,50V, Capacitor_SMD:C_1206_3216Metric, F.Cu at (76.5, 29.0)
- added C35: 2.2uF, Capacitor_SMD:C_0603_1608Metric, F.Cu at (76.2, 10.8)
- added C36: 2.2uF, Capacitor_SMD:C_0603_1608Metric, F.Cu at (76.2, 13.3)
- added C37: 10uF,50V, Capacitor_SMD:C_1206_3216Metric, F.Cu at (3.31, -120.3)
- added C38: 1uF, Capacitor_SMD:C_0402_1005Metric, F.Cu at (-5.02, -126.4)
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Connections:
- C41 pad 1: VDD -> VCC
- C800 pad 2: VDD -> VCC
- D7 pad 1: VDD -> VRAW
- J10 pad 1: INHA -> /VIN
- J10 pad 2: INHB -> GND
- J10 pad 3: INHC -> (no net)
- J7 pad 1: Net-(J7-Pin_1) -> /VIN
- Q7 pad 2: VDD -> VRAW
- Q7 pad 3: Net-(J7-Pin_1) -> /VIN
- R20 pad 1: (no net) -> Net-(D14-K)
- R20 pad 2: (no net) -> V_DETECT
- R33 pad 1: CAN_H -> GND
- R33 pad 2: CAN_L -> /PGND
- R50 pad 1: +3V3 -> Net-(Q10-G)
- R50 pad 2: (no net) -> /IE-FETS-NoOp-B/GHx
- R51 pad 1: (no net) -> Net-(Q11-G)
- R51 pad 2: GND -> /IE-FETS-NoOp-B/GLx
- R62 pad 1: GND -> +3V3
- R62 pad 2: Net-(U60-RES12K) -> sCUR_C2
- R63 pad 1: CHIP_EN -> sCUR_C2
- R63 pad 2: +3V3 -> GND
- R64 pad 1: GPIO2 -> sVLT_C2
- R64 pad 2: +3V3 -> /IE-FETS-NoOp-C/SHx
- R65 pad 1: GPIO0 -> GND
- R65 pad 2: +3V3 -> sVLT_C2
- R9 pad 1: (no net) -> Net-(D14-K)
- R9 pad 2: GND -> Net-(C30-Pad1)
- TP10 pad 1: (no net) -> CC2
- TP2 pad 1: sVLT_B -> Net-(U11-DM)
- TP3 pad 1: sVLT_C -> Net-(U11-DP)
- TP4 pad 1: sCUR_A -> Net-(U11-DEBUG)
- TP5 pad 1: (no net) -> Net-(U11-CC2)
- TP6 pad 1: (no net) -> Net-(U11-CC1)
- TP7 pad 1: (no net) -> /IE-Fets-A/REF_1V65
- TP8 pad 1: sCUR_B -> sCUR_A1
- TP9 pad 1: sCUR_C -> CC1
- U1 pad 4: VDD -> VCC
- U1 pad 5: VDD -> VCC
- U7 pad 42: unconnected-(U7-PB4-Pad42) -> CC2
- U7 pad 44: unconnected-(U7-PB6-Pad44) -> CC1
Routing:
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- removed copper zone on B.Cu, net (none)
- removed copper zone on F.Cu, net (none)
- removed copper zone on In2.Cu, net +3V3
- removed copper zone on B.Cu, net /IE-Fets-A/SHx
- removed copper zone on F.Cu, net /IE-Fets-A/SHx
- removed copper zone on B.Cu, net /IE-Fets-B/SHx
- removed copper zone on F.Cu, net /IE-Fets-B/SHx
- removed copper zone on B.Cu, net /IE-Fets-C/SHx
- removed copper zone on F.Cu, net /IE-Fets-C/SHx
- removed copper zone on B.Cu, net GND
- removed copper zone on In1.Cu, net GND
- removed copper zone on F.Cu, net Net-(J1-Pin_1)
- removed copper zone on F.Cu, net Net-(J2-Pin_1)
- removed copper zone on F.Cu, net Net-(J3-Pin_1)
- removed copper zone on B.Cu, net VDD
Other:
- board size 141 x 82.4 mm -> 64 x 54 mm
- board text added: "1A"
- board text added: "1B"
- board text added: "1C"
- board text added: "2A"
- board text added: "2B"
- board text added: "2C"
- board text added: "IEEE"
- board text added: "INPUT"
- board text added: "OUTPUT"
- board text removed: "3V"
- board text removed: "3V3"
- board text removed: "5V"
- board text removed: "A"
- board text removed: "B"
- board text removed: "C"
- board text removed: "C,D"
- board text removed: "CanH"
- board text removed: "CanL"
- board text removed: "G"
- board text removed: "GND"
- board text removed: "GoldESC V1 © Alfredo Systems 2022"
- board text removed: "H"
- board text removed: "HA"
- board text removed: "HB"
- board text removed: "HC"
- board text removed: "L"
- board text removed: "LA"
- board text removed: "LB"
- board text removed: "LC"
- board text removed: "SWCLK"
- board text removed: "SWDIO"
- board text removed: "VIN"

Commit message: push for 8/8 order
Parts:
- removed C23: 2.2uF, 10V, Capacitor_SMD:C_0402_1005Metric
- removed D1, D2, D3: Z3V3, Diode_SMD:D_SOD-323_HandSoldering
- removed JP4: Fets_Enable2, Connector_PinSocket_2.54mm:PinSocket_1x02_P2.54mm_Vertical
- removed R1, R3: 1mR, Resistor_SMD:R_1206_3216Metric
- removed R10, R11, R12: 15K, Resistor_SMD:R_0402_1005Metric
- removed R13, R14, R15: 2K2, Resistor_SMD:R_0402_1005Metric
- removed R16, R17, R18: 100R, Resistor_SMD:R_0402_1005Metric
- removed R4: 2K, Resistor_SMD:R_0402_1005Metric
- removed R6: 10K, Resistor_SMD:R_0402_1005Metric
- removed R7: 1K, Resistor_SMD:R_0402_1005Metric
- removed TP83, TP84: TestPoint, AlfredoFootprints:GE_TestPoint_Loop
- removed U4, U5, U6: INA185A1, Package_TO_SOT_SMD:SOT-563
- added FB1: BLM15BX601SN1D, Inductor_SMD:L_0402_1005Metric, F.Cu at (-10.5, -10.2)
- added J12: JST SR/SZ, AlfredoFootprints:JST_SH_1x06_Vertical, F.Cu at (-5.90, 14.0)
- added J9: JST SR/SZ, AlfredoFootprints:JST_SH_1x06_Vertical, F.Cu at (-26.0, 14.0)
- C20: value 2.2uF, 10V -> 2.2uF
- C21: value 2.2uF, 10V -> 1uF
- C22: value 2.2uF, 10V -> 10nF
- C7, C8, C9: value 4.7nF -> 0.1uF
- D83: value LED_Red -> LED_Blue
- R2: value 1mR -> 1K; footprint Resistor_SMD:R_1206_3216Metric -> Resistor_SMD:R_0402_1005Metric
- TP1: value TestPoint -> GND
- TP7: value TestPoint -> SWDIO
- TP8: value TestPoint -> SWCLK
- U8: footprint Crystal:Crystal_SMD_5032-4Pin_5.0x3.2mm -> Crystal:Crystal_SMD_3225-4Pin_3.2x2.5mm
- moved C12 198.4 mm to (18.5, 7.68), turned to -90 degrees
- moved C14 196.9 mm to (17.5, 7.68), turned to -90 degrees
- moved C11 195.3 mm to (14.4, 11.4)
- moved U1 193.8 mm to (18.2, 4.54), turned to 90 degrees
- moved C900 193.0 mm to (14.3, 3.00), turned to 180 degrees
- moved C13 192.8 mm to (12.6, 11.4), turned to 180 degrees
- moved R300 191.5 mm to (20.5, 7.68), turned to -90 degrees
- moved C800 191.4 mm to (20.9, 4.00), turned to 90 degrees
- moved R200 190.8 mm to (19.5, 7.68), turned to 90 degrees
- moved U3 189.9 mm to (13.5, 14.3), turned to 90 degrees
- moved L1 185.3 mm to (14.8, 5.80), turned to -90 degrees
- moved R42 175.0 mm to (27.2, -9.50), turned to -90 degrees
- moved R43 175.0 mm to (27.2, -7.50), turned to -90 degrees
- moved C42 172.8 mm to (26.2, -9.49), turned to 90 degrees
- moved D42 153.4 mm to (28.9, -8.50), turned to 90 degrees
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Connections:
- C1 pad 1: VCC -> /IE-FETS-NoOp-A/VFET
- C2 pad 1: VCC -> /IE-FETS-NoOp-A/VFET
- C21 pad 1: +3V3 -> Net-(U7-VDDA)
- C22 pad 1: +3V3 -> Net-(U7-VDDA)
- C3 pad 1: VCC -> /IE-FETS-NoOp-A/VFET
- C41 pad 1: VCC -> /IE-FETS-NoOp-A/VFET
- C43 pad 1: VCC -> /IE-FETS-NoOp-A/VFET
- C44 pad 1: VCC -> /IE-FETS-NoOp-A/VFET
- C7 pad 1: GND -> +3V3
- C7 pad 2: sCUR_A1 -> GND
- C8 pad 1: GND -> +3V3
- C8 pad 2: sCUR_B1 -> GND
- C9 pad 1: GND -> +3V3
- C9 pad 2: sCUR_C1 -> GND
- D11 pad 1: CC1 -> CC2
- D11 pad 2: CC2 -> CC1
- J1 pad 5: /IE-Fets-C/VOUT -> /IE-Fets-C/SHx
- J11 pad 1: /IE-Fets-A/VOUT -> /IE-FETS-NoOp-C/SHx
- J2 pad 1: /IE-Fets-B/VOUT -> /IE-Fets-B/SHx
- J2 pad 2: /IE-Fets-A/VOUT -> /IE-Fets-A/SHx
- J3 pad 2: /IE-Fets-C/VOUT -> /IE-Fets-C/SHx
- J8 pad 3: ENC_A2 -> sCUR_A2_OUT
- J8 pad 4: ENC_B2 -> sCUR_B2_OUT
- J8 pad 5: ENC_C2 -> sCUR_C2_OUT
- JP3 pad 2: /IE-Fets-A/VFET -> /IE-FETS-NoOp-A/VFET
- Q1 pad 5: /IE-Fets-A/VFET -> /IE-FETS-NoOp-A/VFET
- Q2 pad 5: /IE-Fets-A/VFET -> /IE-FETS-NoOp-A/VFET
- Q3 pad 5: /IE-Fets-A/VFET -> /IE-FETS-NoOp-A/VFET
- R2 pad 1: /IE-Fets-B/VOUT -> INHB_1
- R2 pad 2: /IE-Fets-B/SHx -> GND
- R30 pad 1: unconnected-(R30-Pad1) -> +3V3
- R31 pad 1: unconnected-(R31-Pad1) -> STM_LED
- R45 pad 2: sCUR_A2 -> sCUR_A2+
- R46 pad 2: sCUR_A2 -> sCUR_A2+
- R47 pad 1: sCUR_A2 -> sCUR_A2+
- R53 pad 2: sCUR_B2 -> sCUR_B2+
- R54 pad 2: sCUR_B2 -> sCUR_B2+
- R55 pad 1: sCUR_B2 -> sCUR_B2+
- R61 pad 2: sCUR_C2 -> sCUR_C2+
- R62 pad 2: sCUR_C2 -> sCUR_C2+
- R63 pad 1: sCUR_C2 -> sCUR_C2+
- TP1 pad 1: Net-(U7-PB8) -> GND
- TP7 pad 1: /IE-Fets-A/REF_1V65 -> SCL
- TP8 pad 1: sCUR_A1 -> SDA
- U7 pad 10: unconnected-(U7-PA2-Pad10) -> sCUR_A2_OUT
- U7 pad 11: unconnected-(U7-PA3-Pad11) -> GND
- U7 pad 12: unconnected-(U7-PA4-Pad12) -> sVLT_A2
- U7 pad 13: unconnected-(U7-PA5-Pad13) -> GND
- U7 pad 14: unconnected-(U7-PA6-Pad14) -> sCUR_B2_OUT
- U7 pad 15: unconnected-(U7-PA7-Pad15) -> sCUR_B2+
- U7 pad 16: unconnected-(U7-PC4-Pad16) -> sVLT_B2
- U7 pad 17: unconnected-(U7-PB0-Pad17) -> TEMP_FETS
- U7 pad 18: unconnected-(U7-PB1-Pad18) -> sCUR_C2_OUT
- U7 pad 19: unconnected-(U7-PB2-Pad19) -> TEMP_1
- U7 pad 2: unconnected-(U7-PC13-Pad2) -> INLC_2
- U7 pad 20: unconnected-(U7-VREF+-Pad20) -> Net-(U7-VDDA)
- U7 pad 21: +3V3 -> Net-(U7-VDDA)
- U7 pad 22: unconnected-(U7-PB10-Pad22) -> GND
- U7 pad 24: unconnected-(U7-PB11-Pad24) -> sVLT_C2
- U7 pad 25: unconnected-(U7-PB12-Pad25) -> sVLT_VRAW
- U7 pad 26: unconnected-(U7-PB13-Pad26) -> sCUR_C2+
- U7 pad 27: unconnected-(U7-PB14-Pad27) -> INLB_2
- U7 pad 28: unconnected-(U7-PB15-Pad28) -> INLA_2
- U7 pad 29: unconnected-(U7-PC6-Pad29) -> ENC_A1
- U7 pad 3: unconnected-(U7-PC14-Pad3) -> ENC_B1
- U7 pad 30: unconnected-(U7-PA8-Pad30) -> INHC_2
- U7 pad 31: unconnected-(U7-PA9-Pad31) -> INHB_2
- U7 pad 32: unconnected-(U7-PA10-Pad32) -> INHA_2
- U7 pad 33: unconnected-(U7-PA11-Pad33) -> USB_D-
- U7 pad 34: unconnected-(U7-PA12-Pad34) -> USB_D+
- U7 pad 36: unconnected-(U7-PA13-Pad36) -> SCL
- U7 pad 37: unconnected-(U7-PA14-Pad37) -> SDA
- U7 pad 38: unconnected-(U7-PA15-Pad38) -> INHC_1
- U7 pad 39: unconnected-(U7-PC10-Pad39) -> INLC_1
- U7 pad 4: unconnected-(U7-PC15-Pad4) -> ENC_C1
- U7 pad 40: unconnected-(U7-PC11-Pad40) -> INLB_1
- U7 pad 41: unconnected-(U7-PB3-Pad41) -> STM_LED
- U7 pad 43: unconnected-(U7-PB5-Pad43) -> INLA_1
- U7 pad 45: unconnected-(U7-PB7-Pad45) -> lone_dc_encoder_pin
- U7 pad 46: Net-(U7-PB8) -> INHB_1
- U7 pad 47: unconnected-(U7-PB9-Pad47) -> INHA_1
- U7 pad 8: unconnected-(U7-PA0-Pad8) -> TEMP_2
- U7 pad 9: unconnected-(U7-PA1-Pad9) -> sCUR_A2+
Routing:
- net +5V: track 0.00 -> 135.5 mm, vias 0 -> 2
- net TEMP_1: track 0.00 -> 118.8 mm, vias 0 -> 4
- net ENC_A1: track 0.00 -> 118.6 mm, vias 0 -> 2
- net ENC_B1: track 0.00 -> 106.4 mm, vias 0 -> 2
- net TEMP_2: track 0.00 -> 106.1 mm, vias 0 -> 4
- net ENC_C1: track 0.00 -> 105.9 mm, vias 0 -> 2
- net /IE-FETS-NoOp-A/VFET: track 0.00 -> 104.7 mm
- net +3V3: track 0.00 -> 103.0 mm, vias 0 -> 9
- net sCUR_C2_OUT: track 0.00 -> 98.5 mm, vias 0 -> 2
- net sCUR_B2_OUT: track 0.00 -> 95.4 mm, vias 0 -> 2
- net sCUR_A2_OUT: track 0.00 -> 92.2 mm, vias 0 -> 2
- net GND: track 0.00 -> 89.7 mm, vias 0 -> 88
- net /IE-FETS-NoOp-C/SHx: track 0.00 -> 79.2 mm, vias 0 -> 8
- net lone_dc_encoder_pin: track 0.00 -> 78.3 mm, vias 0 -> 3
- net /IE-FETS-NoOp-A/SHx: track 0.00 -> 63.1 mm, vias 0 -> 8
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- added copper zone on In2.Cu, net +3V3
- added copper zone on F.Cu, net /IE-FETS-NoOp-A/SHx
- added copper zone on F.Cu, net /IE-FETS-NoOp-B/SHx
- added copper zone on F.Cu, net /IE-FETS-NoOp-C/SHx
- added copper zone on F.Cu, net /IE-Fets-A/SHx
- added copper zone on F.Cu, net /IE-Fets-B/SHx
- added copper zone on F.Cu, net /IE-Fets-C/SHx
- added copper zone on F.Cu, net GND
- added copper zone on In1.Cu, net GND
- added copper zone on F.Cu, net Net-(Q11-S-Pad1)
- added copper zone on F.Cu, net Net-(Q13-S-Pad1)
- added copper zone on F.Cu, net Net-(Q9-S-Pad1)
- added copper zone on F.Cu, net Net-(U1-LX)
Other:
- board size 64 x 54 mm -> 84 x 54 mm
- board text added: "BOOT"
- board text added: "CC1"
- board text added: "CC2"
- board text added: "DBUG"
- board text added: "DM"
- board text added: "DP"
- board text added: "GND"
- board text added: "L1"
- board text added: "L2"
- board text added: "PB3"
- board text added: "POW"
- board text added: "SCL"
- board text added: "SDA"
- board text added: "VCC"
- board text added: "VCRG"
- board text added: "VFET"
- board text added: "VIN"
- board text added: "VRAW"
- board text added: "Wireless Coil"
- board text removed: "IEEE"

Commit message: first push for v2
Parts:
- C1, C2, C3, C41, C43, C44: value 4.7uF,50V -> 4.7uF, 50V
- C10, C33, C34, C37: value 10uF,50V -> 10uF, 50V
- C13: value 2.2uF, 6.3V -> 2.2uF, 10V
- C15, C16: value 15pF -> 15pF, 50V
- C17, C27, C28, C32, C42, C900: value 100nF -> 100nF, 50V
- C20: value 2.2uF -> 2.2uF, 10V
- C22: value 10nF -> 10nF, 6.3V
- C29: value 250nF -> 250nF, 100V
- C35, C36: value 2.2uF -> 2.2uF, 50V
- C7, C8, C9: value 0.1uF -> 100nF, 50V
- moved H1 0.71 mm to (29.5, 24.5)
- moved H3 0.71 mm to (-38.5, 24.5)
- moved H4 0.71 mm to (29.5, -24.5)
- moved H2 0.50 mm to (-38.5, -18.0)
Connections:
- net S2_EN renamed Net-(U7-PG10)
- C31 pad 1: Net-(C31-Pad1) -> GND
- R34 pad 2: Net-(C31-Pad1) -> GND
- R35 pad 2: Net-(C31-Pad1) -> GND
Routing:
- net GND: track 89.7 -> 91.7 mm
- net Net-(C31-Pad1): track 1.99 -> 0.00 mm
