File: I3ESC.kicad_pcb (KiCad board)
At the start: 4 copper layers, 84 x 54 mm, 169 parts, among them J1 JST SR/SZ, J10 VIN_BARREL, J11 Barrel_Jack, J12 JST SR/SZ, J2 Screw_Terminal_01x02, J3 Screw_Terminal_01x02, J4 Screw_Terminal_01x02, J5 Conn_01x06, J6 Wireless Coil, J7 VIN_TERMINAL, J8 Conn_01x06, J9 JST SR/SZ, Q1 YJG150N03A, Q10 YJG150N03A, Q11 YJG150N03A, Q12 YJG150N03A, Q13 YJG150N03A, Q2 YJG150N03A, Q3 YJG150N03A, Q4 YJG150N03A, Q5 YJG150N03A, Q6 YJG150N03A, Q7 AO3401A, Q8 YJG150N03A, Q9 YJG150N03A, SW1 reset, U1 SY8113BADC, U10 USBLC6-2P6, U11 IP6826, U12 FD8288T (DRV8300), U13 Qwiic1, U2 FD8288T (DRV8300), U3 SPX3819M5-L-3-3, U7 STM32G431CBUx, U8 ABM3B-8.000MHZ, U9 USB_C_Receptacle

Commit message: big schematic push for stm32g474
Parts:
- removed Q10, Q11, Q12, Q13, Q8, Q9: YJG150N03A, Package_TO_SOT_SMD:LFPAK56
- removed Q7: AO3401A, AlfredoFootprints:SOT-23-small
- removed U7: STM32G431CBUx, Package_DFN_QFN:QFN-48-1EP_7x7mm_P0.5mm_EP5.6x5.6mm
- added C23: 100nF, 50V, Capacitor_SMD:C_0402_1005Metric, F.Cu at (-107.3, -18.7)
- added C45: 100nF, 50V, Capacitor_SMD:C_0402_1005Metric, F.Cu at (-85.0, -25.3)
- added C46: 100nF, 50V, Capacitor_SMD:C_0402_1005Metric, F.Cu at (-107.3, -16.7)
- added D1: Z3V3, Diode_SMD:D_SOD-523, F.Cu at (-76.0, 23.4)
- added D2: Z3V3, Diode_SMD:D_SOD-523, F.Cu at (-101.8, -44.7)
- added D3: Z3V3, Diode_SMD:D_SOD-523, F.Cu at (-86.2, -44.7)
- added R1: 10R, Resistor_SMD:R_0402_1005Metric, F.Cu at (-85.1, -11.2)
- added R10: 10R, Resistor_SMD:R_0402_1005Metric, F.Cu at (-64.4, -9.19)
- added R11: 10R, Resistor_SMD:R_0402_1005Metric, F.Cu at (-106.8, 2.20)
- added R12: 10R, Resistor_SMD:R_0402_1005Metric, F.Cu at (-106.8, 3.60)
- added R13: 2mR, Resistor_SMD:R_1206_3216Metric, F.Cu at (-79.4, 14.8)
- added R14: 22K, Resistor_SMD:R_0402_1005Metric, F.Cu at (-75.5, 20.1)
- added R15: 2K2, Resistor_SMD:R_0402_1005Metric, F.Cu at (-76.5, 20.1)
- added R16: 2K2, Resistor_SMD:R_0402_1005Metric, F.Cu at (-76.0, 18.7)
- added R17: 15K, Resistor_SMD:R_0402_1005Metric, F.Cu at (-75.5, 21.9)
- added R18: 2K2, Resistor_SMD:R_0402_1005Metric, F.Cu at (-76.5, 21.9)
- added R3: 10R, Resistor_SMD:R_0402_1005Metric, F.Cu at (-85.1, -9.19)
- added R32: 15K, Resistor_SMD:R_0402_1005Metric, F.Cu at (-111.5, -42.0)
- added R36: 2K2, Resistor_SMD:R_0402_1005Metric, F.Cu at (-111.5, -40.0)
- added R37: 10R, Resistor_SMD:R_0402_1005Metric, F.Cu at (-95.8, -52.0)
- added R4: 10R, Resistor_SMD:R_0402_1005Metric, F.Cu at (-74.7, -11.2)
- added R6: 10R, Resistor_SMD:R_0402_1005Metric, F.Cu at (-74.7, -9.19)
- added R66: 2K2, Resistor_SMD:R_0402_1005Metric, F.Cu at (-95.8, -40.0)
- added R67: 1K, Resistor_SMD:R_0402_1005Metric, F.Cu at (-84.9, -27.3)
- added R7: 10R, Resistor_SMD:R_0402_1005Metric, F.Cu at (-64.4, -11.2)
- added SW2: boot, AlfredoFootprints:Button_SKRKAEE020, F.Cu at (-105.6, -21.7)
- added SW3: user1, AlfredoFootprints:Button_SKRKAEE020, F.Cu at (-69.0, -29.3)
- added U4: STM32G474RETx, Package_QFP:LQFP-64_10x10mm_P0.5mm, F.Cu at (-35.0, -47.0)
- added U5: Qwiic1, Connector_JST:JST_SH_BM04B-SRSS-TB_1x04-1MP_P1.00mm_Vertical, F.Cu at (-54.9, -49.4)
- D18, D19, D20, D42: footprint Diode_SMD:D_SOD-323_HandSoldering -> Diode_SMD:D_SOD-523
- D7: value Z5V6 -> LED_RED; footprint AlfredoFootprints:D_SOD-323 -> LED_SMD:LED_0603_1608Metric
- Q1, Q2, Q3, Q4, Q5, Q6: value YJG150N03A -> ~; footprint Package_TO_SOT_SMD:LFPAK56 -> AlfredoFootprints:DFN-8-2EP_6x5mm
- R22, R39: value 10R -> 2mR; footprint Resistor_SMD:R_0402_1005Metric -> Resistor_SMD:R_1206_3216Metric
- R23, R50: value 10R -> 22K
- R24, R25, R51, R58: value 10R -> 2K2
- R44, R52, R60: value 1mR -> 2mR
- R5: value 10K -> 1K
- R59: value 10R -> 15K
- moved D7 128.7 mm to (-103.8, -18.3), turned to 0 degrees
- moved R5 127.8 mm to (-101.0, -20.8), turned to 0 degrees
- moved R58 104.3 mm to (-95.8, -44.0), turned to 0 degrees
- moved R59 100.2 mm to (-95.8, -42.0), turned to 0 degrees
- moved R50 99.2 mm to (-95.8, -48.0), turned to 0 degrees
- moved C2 96.0 mm to (-107.2, -44.5), turned to 0 degrees
- moved R51 94.4 mm to (-95.8, -46.0), turned to 0 degrees
- moved R38 93.5 mm to (-95.8, -50.0), turned to 0 degrees
- moved Q1 89.4 mm to (-105.4, -49.5), turned to 0 degrees
- moved R23 88.2 mm to (-111.5, -48.0), turned to 0 degrees
- moved R19 87.9 mm to (-111.5, -52.0), turned to 0 degrees
- moved R25 86.0 mm to (-111.5, -44.0), turned to 0 degrees
- moved R21 84.3 mm to (-111.5, -50.0), turned to 0 degrees
- moved R24 83.8 mm to (-111.5, -46.0), turned to 0 degrees
- moved C3 83.4 mm to (-91.6, -44.5), turned to 0 degrees
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Connections:
- net TEMP_FETS renamed OPAMP3_VOUT
- net sVLT_A2 renamed sVLT_2A
- net sVLT_B2 renamed sVLT_2B
- net sVLT_C2 renamed sVLT_2C
- C1 pad 1: /IE-FETS-NoOp-A/VFET -> /IE-FETS-1A/VFET
- C2 pad 1: /IE-FETS-NoOp-A/VFET -> /IE-FETS-1A/VFET
- C21 pad 1: Net-(U7-VDDA) -> +3V3
- C22 pad 1: Net-(U7-VDDA) -> +3V3
- C3 pad 1: /IE-FETS-NoOp-A/VFET -> /IE-FETS-1A/VFET
- C38 pad 2: /IE-FETS-NoOp-A/SHx -> /IE-FETS-2A/SHx
- C39 pad 2: /IE-FETS-NoOp-B/SHx -> /IE-FETS-2B/SHx
- C4 pad 2: /IE-Fets-A/SHx -> /IE-FETS-1A/SHx
- C40 pad 2: /IE-FETS-NoOp-C/SHx -> /IE-FETS-2C/SHx
- C41 pad 1: /IE-FETS-NoOp-A/VFET -> /IE-FETS-1A/VFET
- C43 pad 1: /IE-FETS-NoOp-A/VFET -> /IE-FETS-1A/VFET
- C44 pad 1: /IE-FETS-NoOp-A/VFET -> /IE-FETS-1A/VFET
- C5 pad 2: /IE-Fets-B/SHx -> /IE-FETS-1B/SHx
- C6 pad 2: /IE-Fets-C/SHx -> /IE-FETS-1C/SHx
- D7 pad 1: VRAW -> GND
- FB1 pad 2: Net-(U7-VDDA) -> +3V3
- J1 pad 5: /IE-Fets-C/SHx -> /IE-FETS-1C/SHx
- J1 pad 6: /IE-FETS-NoOp-A/SHx -> /IE-FETS-2A/SHx
- J10 pad 1: /VIN -> VRAW
- J11 pad 1: /IE-FETS-NoOp-C/SHx -> /IE-FETS-2B/SHx
- J11 pad 2: GND -> /IE-FETS-2C/SHx
- J12 pad 5: /IE-FETS-NoOp-B/SHx -> /IE-FETS-2B/SHx
- J12 pad 6: /IE-FETS-NoOp-C/SHx -> /IE-FETS-2C/SHx
- J2 pad 1: /IE-Fets-B/SHx -> /IE-FETS-1B/SHx
- J2 pad 2: /IE-Fets-A/SHx -> /IE-FETS-1A/SHx
- J3 pad 1: /IE-FETS-NoOp-A/SHx -> /IE-FETS-2A/SHx
- J3 pad 2: /IE-Fets-C/SHx -> /IE-FETS-1C/SHx
- J4 pad 1: /IE-FETS-NoOp-C/SHx -> /IE-FETS-2C/SHx
- J4 pad 2: /IE-FETS-NoOp-B/SHx -> /IE-FETS-2B/SHx
- J7 pad 1: /VIN -> VRAW
- J9 pad 5: /IE-Fets-A/SHx -> /IE-FETS-1A/SHx
- J9 pad 6: /IE-Fets-B/SHx -> /IE-FETS-1B/SHx
- JP3 pad 2: /IE-FETS-NoOp-A/VFET -> /IE-FETS-1A/VFET
- Q1 pad 1: /IE-Fets-A/SHx -> unconnected-(Q1-S1-Pad1)
- Q1 pad 2: /IE-Fets-A/SHx -> Net-(Q1-G1)
- Q1 pad 3: /IE-Fets-A/SHx -> Net-(Q1-S2)
- Q1 pad 4: Net-(Q1-G) -> Net-(Q1-G2)
- Q1 pad 5: /IE-FETS-NoOp-A/VFET -> /IE-FETS-1B/SHx
- Q2 pad 1: /IE-Fets-B/SHx -> unconnected-(Q2-S1-Pad1)
- Q2 pad 2: /IE-Fets-B/SHx -> Net-(Q2-G1)
- Q2 pad 3: /IE-Fets-B/SHx -> Net-(Q2-S2)
- Q2 pad 4: Net-(Q2-G) -> Net-(Q2-G2)
- Q2 pad 5: /IE-FETS-NoOp-A/VFET -> /IE-FETS-1C/SHx
- Q3 pad 1: /IE-Fets-C/SHx -> unconnected-(Q3-S1-Pad1)
- Q3 pad 2: /IE-Fets-C/SHx -> Net-(Q3-G1)
- Q3 pad 3: /IE-Fets-C/SHx -> Net-(Q3-S2)
- Q3 pad 4: Net-(Q3-G) -> Net-(Q3-G2)
- Q3 pad 5: /IE-FETS-NoOp-A/VFET -> /IE-FETS-2A/SHx
- Q4 pad 1: GND -> unconnected-(Q4-S1-Pad1)
- Q4 pad 2: GND -> Net-(Q4-G1)
- Q4 pad 3: GND -> Net-(Q4-S2)
- Q4 pad 4: Net-(Q4-G) -> Net-(Q4-G2)
- Q4 pad 5: /IE-Fets-A/SHx -> /IE-FETS-1A/SHx
- Q5 pad 1: GND -> unconnected-(Q5-S1-Pad1)
- Q5 pad 2: GND -> Net-(Q5-G1)
- Q5 pad 3: GND -> Net-(Q5-S2)
- Q5 pad 4: Net-(Q5-G) -> Net-(Q5-G2)
- Q5 pad 5: /IE-Fets-B/SHx -> /IE-FETS-2B/SHx
- Q6 pad 1: GND -> unconnected-(Q6-S1-Pad1)
- Q6 pad 2: GND -> Net-(Q6-G1)
- Q6 pad 3: GND -> Net-(Q6-S2)
- Q6 pad 4: Net-(Q6-G) -> Net-(Q6-G2)
- Q6 pad 5: /IE-Fets-C/SHx -> /IE-FETS-2C/SHx
- R19 pad 1: Net-(Q1-G) -> Net-(Q1-G1)
- R19 pad 2: /IE-Fets-A/GHx -> /IE-FETS-1B/GHx
- R2 pad 1: INHB_1 -> BOOT
- R21 pad 1: Net-(Q4-G) -> Net-(Q1-G2)
- R21 pad 2: /IE-Fets-A/GLx -> /IE-FETS-1B/GLx
- R22 pad 1: Net-(Q2-G) -> Net-(Q1-S2)
- R22 pad 2: /IE-Fets-B/GHx -> GND
- R23 pad 1: Net-(Q5-G) -> +3V3
- R23 pad 2: /IE-Fets-B/GLx -> Net-(Q1-S2)
- R24 pad 1: Net-(Q3-G) -> Net-(Q1-S2)
- R24 pad 2: /IE-Fets-C/GHx -> GND
- R25 pad 1: Net-(Q6-G) -> Net-(Q1-S2)
- R25 pad 2: /IE-Fets-C/GLx -> /IE-FETS-1B/sCURx+
- R31 pad 1: STM_LED -> STM_LED1
- R38 pad 1: Net-(Q8-G) -> Net-(Q2-G2)
- R38 pad 2: /IE-FETS-NoOp-A/GHx -> /IE-FETS-1C/GLx
- R39 pad 1: Net-(Q9-G) -> Net-(Q2-S2)
- R39 pad 2: /IE-FETS-NoOp-A/GLx -> GND
- R44 pad 1: Net-(Q9-S-Pad1) -> Net-(Q3-S2)
- R45 pad 1: Net-(Q9-S-Pad1) -> Net-(Q3-S2)
- R45 pad 2: sCUR_A2+ -> /IE-FETS-2A/sCURx+
- R46 pad 2: sCUR_A2+ -> Net-(Q3-S2)
- R47 pad 1: sCUR_A2+ -> Net-(Q3-S2)
- R48 pad 2: /IE-FETS-NoOp-A/SHx -> /IE-FETS-2A/SHx
- R5 pad 1: Net-(D7-A) -> STM_LED2
- R5 pad 2: GND -> Net-(D7-A)
- R50 pad 1: Net-(Q10-G) -> +3V3
- R50 pad 2: /IE-FETS-NoOp-B/GHx -> Net-(Q2-S2)
- R51 pad 1: Net-(Q11-G) -> Net-(Q2-S2)
- R51 pad 2: /IE-FETS-NoOp-B/GLx -> GND
- R52 pad 1: Net-(Q11-S-Pad1) -> Net-(Q5-S2)
- R53 pad 1: Net-(Q11-S-Pad1) -> Net-(Q5-S2)
- R53 pad 2: sCUR_B2+ -> /IE-FETS-2B/sCURx+
- R54 pad 2: sCUR_B2+ -> Net-(Q5-S2)
- R55 pad 1: sCUR_B2+ -> Net-(Q5-S2)
- R56 pad 2: /IE-FETS-NoOp-B/SHx -> /IE-FETS-2B/SHx
- R58 pad 1: Net-(Q12-G) -> Net-(Q2-S2)
- R58 pad 2: /IE-FETS-NoOp-C/GHx -> /IE-FETS-1C/sCURx+
- R59 pad 1: Net-(Q13-G) -> sVLT_1C
- R59 pad 2: /IE-FETS-NoOp-C/GLx -> /IE-FETS-1C/SHx
- R60 pad 1: Net-(Q13-S-Pad1) -> Net-(Q6-S2)
- R61 pad 1: Net-(Q13-S-Pad1) -> Net-(Q6-S2)
- R61 pad 2: sCUR_C2+ -> /IE-FETS-2C/sCURx+
- R62 pad 2: sCUR_C2+ -> Net-(Q6-S2)
- R63 pad 1: sCUR_C2+ -> Net-(Q6-S2)
- R64 pad 2: /IE-FETS-NoOp-C/SHx -> /IE-FETS-2C/SHx
- TP7 pad 1: SCL -> SWDIO
- TP8 pad 1: SDA -> SWCLK
- U12 pad 1: INHA_2 -> IN_H_2A
- U12 pad 10: /IE-FETS-NoOp-B/GLx -> /IE-FETS-2B/GLx
- U12 pad 11: /IE-FETS-NoOp-A/GLx -> /IE-FETS-2A/GLx
- U12 pad 12: /IE-FETS-NoOp-C/SHx -> /IE-FETS-2C/SHx
- U12 pad 13: /IE-FETS-NoOp-C/GHx -> /IE-FETS-2C/GHx
- U12 pad 15: /IE-FETS-NoOp-B/SHx -> /IE-FETS-2B/SHx
- U12 pad 16: /IE-FETS-NoOp-B/GHx -> /IE-FETS-2B/GHx
- U12 pad 18: /IE-FETS-NoOp-A/SHx -> /IE-FETS-2A/SHx
- U12 pad 19: /IE-FETS-NoOp-A/GHx -> /IE-FETS-2A/GHx
- U12 pad 2: INHB_2 -> IN_H_2B
- U12 pad 3: INHC_2 -> IN_H_2C
- U12 pad 4: INLA_2 -> IN_L_2A
- U12 pad 5: INLB_2 -> IN_L_2B
- U12 pad 6: INLC_2 -> IN_L_2C
- U12 pad 9: /IE-FETS-NoOp-C/GLx -> /IE-FETS-2C/GLx
- U2 pad 1: INHA_1 -> IN_H_1A
- U2 pad 10: /IE-Fets-B/GLx -> /IE-FETS-1B/GLx
- U2 pad 11: /IE-Fets-A/GLx -> /IE-FETS-1A/GLx
- U2 pad 12: /IE-Fets-C/SHx -> /IE-FETS-1C/SHx
- U2 pad 13: /IE-Fets-C/GHx -> /IE-FETS-1C/GHx
- U2 pad 15: /IE-Fets-B/SHx -> /IE-FETS-1B/SHx
- U2 pad 16: /IE-Fets-B/GHx -> /IE-FETS-1B/GHx
- U2 pad 18: /IE-Fets-A/SHx -> /IE-FETS-1A/SHx
- U2 pad 19: /IE-Fets-A/GHx -> /IE-FETS-1A/GHx
- U2 pad 2: INHB_1 -> IN_H_1B
- U2 pad 3: INHC_1 -> IN_H_1C
- U2 pad 4: INLA_1 -> IN_L_1A
- U2 pad 5: INLB_1 -> IN_L_1B
- U2 pad 6: INLC_1 -> IN_L_1C
- U2 pad 9: /IE-Fets-C/GLx -> /IE-FETS-1C/GLx
Routing:
- net (no net): track 0.00 -> 278.9 mm, vias 0 -> 26
- net /IE-FETS-NoOp-A/VFET: track 104.7 -> 0.00 mm
- net /IE-FETS-1A/VFET: track 0.00 -> 104.7 mm
- net /IE-FETS-NoOp-C/SHx: track 79.2 -> 0.00 mm, vias 8 -> 0
- net /IE-FETS-NoOp-A/SHx: track 63.1 -> 0.00 mm, vias 8 -> 0
- net /IE-FETS-2A/SHx: track 0.00 -> 63.1 mm, vias 0 -> 8
- net /IE-FETS-NoOp-B/SHx: track 57.3 -> 0.00 mm, vias 8 -> 0
- net /IE-FETS-2B/SHx: track 0.00 -> 57.3 mm, vias 0 -> 8
- net /IE-Fets-C/SHx: track 55.6 -> 0.00 mm, vias 9 -> 0
- net /IE-FETS-1C/SHx: track 0.00 -> 55.6 mm, vias 0 -> 9
- net /IE-Fets-B/SHx: track 47.0 -> 0.00 mm, vias 8 -> 0
- net /IE-FETS-1B/SHx: track 0.00 -> 47.0 mm, vias 0 -> 8
- net /IE-Fets-A/SHx: track 44.4 -> 0.00 mm, vias 8 -> 0
- net /IE-FETS-1A/SHx: track 0.00 -> 44.4 mm, vias 0 -> 8
- net /IE-FETS-NoOp-A/GHx: track 36.5 -> 0.00 mm, vias 2 -> 0
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- added copper zone on F.Cu, net /IE-FETS-1A/SHx
- added copper zone on F.Cu, net /IE-FETS-1B/SHx
- added copper zone on F.Cu, net /IE-FETS-1C/SHx
- added copper zone on F.Cu, net /IE-FETS-2A/SHx
- added copper zone on F.Cu, net /IE-FETS-2B/SHx
- added copper zone on F.Cu, net /IE-FETS-2C/SHx
- added copper zone on F.Cu, net Net-(Q3-S2)
- added copper zone on F.Cu, net Net-(Q5-S2)
- added copper zone on F.Cu, net Net-(Q6-S2)
- removed copper zone on F.Cu, net /IE-FETS-NoOp-A/SHx
- removed copper zone on F.Cu, net /IE-FETS-NoOp-B/SHx
- removed copper zone on F.Cu, net /IE-FETS-NoOp-C/SHx
- removed copper zone on F.Cu, net /IE-Fets-A/SHx
- removed copper zone on F.Cu, net /IE-Fets-B/SHx
- removed copper zone on F.Cu, net /IE-Fets-C/SHx
- removed copper zone on F.Cu, net Net-(Q11-S-Pad1)
- removed copper zone on F.Cu, net Net-(Q13-S-Pad1)
- removed copper zone on F.Cu, net Net-(Q9-S-Pad1)
Other:
- board size 84 x 54 mm -> 84 x 111 mm
- board text added: "RST"
- board text removed: "BOOT"

Commit message: huge layout progress
Parts:
- removed C17: 100nF, 50V, Capacitor_SMD:C_0402_1005Metric
- removed C19: 220uF, Capacitor_SMD:CP_Elec_6.3x7.7
- removed JP3: Fets_Enable1, Connector_PinSocket_2.54mm:PinSocket_1x02_P2.54mm_Vertical
- removed SW1: reset, AlfredoFootprints:Button_SKRKAEE020
- removed TP10: TP_CC2, AlfredoFootprints:GE_TestPoint_Loop
- removed TP3: TP_DP, AlfredoFootprints:GE_TestPoint_Loop
- removed TP7: SWDIO, AlfredoFootprints:GE_TestPoint_Loop
- removed TP8: SWCLK, AlfredoFootprints:GE_TestPoint_Loop
- removed TP9: TP_CC1, AlfredoFootprints:GE_TestPoint_Loop
- removed U13: Qwiic1, Connector_JST:JST_SH_BM04B-SRSS-TB_1x04-1MP_P1.00mm_Vertical
- added J13: Conn_01x04, Connector_PinHeader_2.54mm:PinHeader_1x04_P2.54mm_Vertical, B.Cu at (-24.9, -25.3)
- added JP4: Qi_D-, Connector_PinSocket_2.54mm:PinSocket_1x02_P2.54mm_Vertical, F.Cu at (34.3, -5.08)
- added JP5: Qi_D+, Connector_PinSocket_2.54mm:PinSocket_1x02_P2.54mm_Vertical, F.Cu at (36.8, -5.08)
- added JP6: Qi_CC2, Connector_PinSocket_2.54mm:PinSocket_1x02_P2.54mm_Vertical, F.Cu at (39.4, -2.54)
- added JP7: Qi_CC1, Connector_PinSocket_2.54mm:PinSocket_1x02_P2.54mm_Vertical, F.Cu at (31.8, -5.08)
- added U6: USB_C_Receptacle, AlfredoFootprints:USB_TYPE-C-31-M-12, F.Cu at (37.1, -14.0)
- JP2: value VRAW to VCC -> VCC-bypass; footprint Connector_PinSocket_2.54mm:PinSocket_1x02_P2.54mm_Vertical -> AlfredoFootprints:SolderJumper-2-Small; moved to B.Cu
- SW2: value boot -> boot-red; footprint AlfredoFootprints:Button_SKRKAEE020 -> AlfredoFootprints:button-3.6x6mm
- SW3: value user1 -> user1-white; footprint AlfredoFootprints:Button_SKRKAEE020 -> AlfredoFootprints:button-3.6x6mm
- TP2: value TP_DM -> QI_PGND
- moved R23 110.3 mm to (-14.5, 4.60), turned to 90 degrees
- moved R24 108.5 mm to (-15.5, 4.60), turned to -90 degrees
- moved R32 108.4 mm to (-14.5, 6.40), turned to 90 degrees
- moved C46 108.0 mm to (0.30, -7.60), turned to -135 degrees
- moved R25 107.4 mm to (-15.0, 3.20)
- moved R36 106.6 mm to (-15.5, 6.40), turned to -90 degrees
- moved Q5 104.8 mm to (5.00, 4.50), turned to -90 degrees
- moved R50 103.7 mm to (-6.50, 4.60), turned to 90 degrees
- moved C2 102.6 mm to (-15.0, 0.40), turned to 90 degrees
- moved R21 101.9 mm to (-21.1, -2.90), turned to 90 degrees
- moved Q1 101.9 mm to (-19.0, 4.50), turned to -90 degrees
- moved R51 101.8 mm to (-7.50, 4.60), turned to -90 degrees
- moved R59 101.6 mm to (-6.50, 6.40), turned to 90 degrees
- moved D2 101.5 mm to (-15.0, 7.90), turned to 180 degrees
- moved R19 100.9 mm to (-23.3, -2.90), turned to 90 degrees
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Connections:
- C1 pad 1: /IE-FETS-1A/VFET -> VCC
- C18 pad 1: VRAW -> VCC
- C2 pad 1: /IE-FETS-1A/VFET -> VCC
- C21 pad 1: +3V3 -> Net-(U4-VDDA)
- C22 pad 1: +3V3 -> Net-(U4-VDDA)
- C3 pad 1: /IE-FETS-1A/VFET -> VCC
- C41 pad 1: /IE-FETS-1A/VFET -> VCC
- C43 pad 1: /IE-FETS-1A/VFET -> VCC
- C44 pad 1: /IE-FETS-1A/VFET -> VCC
- FB1 pad 2: +3V3 -> Net-(U4-VDDA)
- J1 pad 2: ENC_B1 -> ENC_2A
- J1 pad 3: ENC_A1 -> ENC_1C
- J10 pad 1: VRAW -> VCC
- J12 pad 2: TEMP_1 -> ENC_2C
- J12 pad 3: TEMP_2 -> ENC_2B
- J5 pad 3: ENC_A1 -> ENC_1C
- J5 pad 4: ENC_B1 -> ENC_1B
- J5 pad 5: ENC_C1 -> ENC_1A
- J7 pad 1: VRAW -> VCC
- J8 pad 3: sCUR_A2_OUT -> ENC_2C
- J8 pad 4: sCUR_B2_OUT -> ENC_2B
- J8 pad 5: sCUR_C2_OUT -> ENC_2A
- J9 pad 2: ENC_C1 -> ENC_1B
- J9 pad 3: lone_dc_encoder_pin -> ENC_1A
- JP1 pad 1: VRAW -> /V_QI_USB
- JP2 pad 2: VRAW -> /V_USB
- Q1 pad 6: /IE-FETS-1A/VFET -> VCC
- Q2 pad 6: /IE-FETS-1A/VFET -> VCC
- Q3 pad 6: /IE-FETS-1A/VFET -> VCC
- Q4 pad 6: /IE-FETS-1A/VFET -> VCC
- Q5 pad 6: /IE-FETS-1A/VFET -> VCC
- Q6 pad 6: /IE-FETS-1A/VFET -> VCC
- R16 pad 2: /IE-FETS-1A/sCURx+ -> OPAMP1_V+
- R25 pad 2: /IE-FETS-1B/sCURx+ -> OPAMP2_V+
- R40 pad 1: +5V -> +3V3
- R43 pad 2: VRAW -> VCC
- R45 pad 2: /IE-FETS-2A/sCURx+ -> OPAMP4_V+
- R53 pad 2: /IE-FETS-2B/sCURx+ -> OPAMP5_V+
- R58 pad 2: /IE-FETS-1C/sCURx+ -> OPAMP3_V+
- R61 pad 2: /IE-FETS-2C/sCURx+ -> OPAMP4_VOUT
- TP2 pad 1: Net-(U11-DM) -> /PGND
- U11 pad 28: Net-(U11-DM) -> Net-(JP4-B)
- U4 pad 28: +3V3 -> Net-(U4-VDDA)
- U4 pad 29: +3V3 -> Net-(U4-VDDA)
- U4 pad 39: STM_LED1 -> STM_LED2
- U4 pad 44: STM_LED2 -> STM_LED1
Routing:
- net (no net): track 278.9 -> 0.00 mm, vias 26 -> 0
- net +5V: track 135.5 -> 0.00 mm, vias 2 -> 0
- net TEMP_1: track 118.8 -> 0.00 mm, vias 4 -> 0
- net ENC_A1: track 118.6 -> 0.00 mm, vias 2 -> 0
- net +3V3: track 108.7 -> 0.70 mm, vias 9 -> 1
- net ENC_B1: track 106.4 -> 0.00 mm, vias 2 -> 0
- net TEMP_2: track 106.1 -> 0.00 mm, vias 4 -> 0
- net ENC_C1: track 105.9 -> 0.00 mm, vias 2 -> 0
- net /IE-FETS-1A/VFET: track 104.7 -> 0.00 mm
- net sCUR_C2_OUT: track 98.5 -> 0.00 mm, vias 2 -> 0
- net sCUR_B2_OUT: track 95.4 -> 0.00 mm, vias 2 -> 0
- net sCUR_A2_OUT: track 92.2 -> 0.00 mm, vias 2 -> 0
- net GND: track 91.7 -> 12.5 mm, vias 88 -> 12
- net lone_dc_encoder_pin: track 78.3 -> 0.00 mm, vias 3 -> 0
- net VRAW: track 65.5 -> 0.00 mm
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- added copper zone on F.Cu, net Net-(Q1-S2)
- added copper zone on F.Cu, net Net-(Q2-S2)
- added copper zone on F.Cu, net Net-(Q4-S2)
- added copper zone on F.Cu, net VCC
- removed copper zone on F.Cu, net /IE-FETS-1A/SHx
- removed copper zone on F.Cu, net /IE-FETS-1B/SHx
- removed copper zone on F.Cu, net /IE-FETS-1C/SHx
- removed copper zone on F.Cu, net /IE-FETS-2A/SHx
- removed copper zone on F.Cu, net /IE-FETS-2B/SHx
- removed copper zone on F.Cu, net /IE-FETS-2C/SHx
Other:
- board size 84 x 111 mm -> 74 x 111 mm
- board text added: "BOOT"
- board text added: "MODE"
- board text added: "PA10"
- board text added: "PC7"
- board text added: "QWIIC"
- board text removed: "L1"
- board text removed: "L2"
- board text removed: "PB3"
- board text removed: "RST"
- board text removed: "SCL"
- board text removed: "SDA"
- board text removed: "VCC"
- board text removed: "VCRG"
- board text removed: "VFET"
- board text removed: "VRAW"

Commit message: majority of routing for V2 completed
Parts:
- added TP3: RST, AlfredoFootprints:GE_TestPoint_Loop, F.Cu at (50.1, -37.7)
- moved C11 62.9 mm to (-43.3, 0.00)
- moved C13 62.9 mm to (-43.3, 1.90)
- moved U3 62.9 mm to (-40.5, 0.95)
- moved C26 14.8 mm to (3.30, -31.2)
- moved D13 14.8 mm to (1.90, -31.0)
- moved R6 14.6 mm to (-4.70, -2.40), turned to 0 degrees
- moved D8 14.4 mm to (7.20, -30.3)
- moved U10 14.1 mm to (-0.70, -30.9), turned to 90 degrees
- moved C37 11.6 mm to (16.4, -8.40), turned to -90 degrees
- moved R4 8.71 mm to (-2.10, -2.40), turned to 0 degrees
- moved JP2 6.51 mm to (1.20, -28.8)
- moved R40 5.92 mm to (-9.50, -3.00)
- moved R41 5.92 mm to (-8.40, -3.00)
- moved R8 5.73 mm to (-11.6, -3.10), turned to -135 degrees
- moved R10 5.02 mm to (10.5, -2.40), turned to 180 degrees
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Connections:
- J5 pad 2: TEMP_1 -> OPAMP1_VOUT
- R40 pad 2: OPAMP3_VOUT -> OPAMP2_VOUT
- R41 pad 1: OPAMP3_VOUT -> OPAMP2_VOUT
- U4 pad 12: sVLT_VRAW -> sVLT_1B
- U4 pad 17: sVLT_1A -> sVLT_1C
- U4 pad 18: sVLT_1B -> sVLT_2A
- U4 pad 19: sVLT_1C -> sVLT_2B
- U4 pad 26: sVLT_2B -> sVLT_2C
- U4 pad 43: sVLT_2A -> sVLT_VRAW
- U4 pad 8: sVLT_2C -> sVLT_1A
Routing:
- net +3V3: track 0.70 -> 110.1 mm, vias 1 -> 13
- net ENC_1C: track 0.00 -> 61.3 mm, vias 0 -> 1
- net ENC_1A: track 0.00 -> 59.4 mm, vias 0 -> 1
- net /IE-FETS-1C/SHx: track 0.00 -> 56.0 mm, vias 0 -> 14
- net /IE-FETS-2A/SHx: track 0.00 -> 54.1 mm, vias 0 -> 14
- net ENC_1B: track 0.00 -> 52.4 mm, vias 0 -> 1
- net USER1: track 0.00 -> 50.7 mm, vias 0 -> 2
- net /IE-FETS-2B/SHx: track 0.00 -> 48.5 mm, vias 0 -> 14
- net /IE-FETS-1A/SHx: track 0.70 -> 49.2 mm, vias 1 -> 14
- net /IE-FETS-1B/SHx: track 0.00 -> 46.9 mm, vias 0 -> 14
- net OPAMP1_VOUT: track 0.00 -> 40.9 mm, vias 0 -> 1
- net /IE-FETS-2C/SHx: track 0.00 -> 40.7 mm, vias 0 -> 14
- net sVLT_2C: track 2.07 -> 41.1 mm, vias 0 -> 2
- net GND: track 12.5 -> 50.7 mm, vias 12 -> 99
- net sVLT_VRAW: track 0.00 -> 34.9 mm
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Other:
- board size 74 x 111 mm -> 74 x 54 mm
