File: I3ESC.kicad_pcb (KiCad board)
At the start: 4 copper layers, 64 x 54 mm, 154 parts, among them J1 JST SR/SZ, J10 VIN_BARREL, J12 JST SR/SZ, J2 Screw_Terminal_01x02, J3 Screw_Terminal_01x02, J4 Screw_Terminal_01x02, J5 Encoder1, J6 5V out, J7 VIN_TERMINAL, J8 Encoder2, J9 JST SR/SZ, SW1 reset, SW2 boot-red, SW3 user1-white, U1 SY8113BADC, U10 USBLC6-2P6, U11 Qwiic2, U12 FD8288T (DRV8300), U2 FD8288T (DRV8300), U3 SPX3819M5-L-3-3, U4 STM32G474RETx, U5 Qwiic1, U7 Prog, U8 ABM3B-8.000MHZ, U9 USB_C_Receptacle

Commit message: updates for production run 2
Parts:
- removed U7: Prog, Connector_JST:JST_SH_BM04B-SRSS-TB_1x04-1MP_P1.00mm_Vertical
- added J11: VIN_BARREL, AlfredoFootprints:DC-005C_1, F.Cu at (20.5, 24.3)
- added J13: Conn_01x03, AlfredoFootprints:PinHeader_1x03_P2.54mm_Vertical, F.Cu at (28.9, -9.68)
- moved C800 22.2 mm to (29.8, 19.9), turned to 0 degrees
- moved R300 20.9 mm to (26.1, 19.5), turned to 180 degrees
- moved R200 18.9 mm to (26.1, 18.5), turned to 0 degrees
- moved J6 17.4 mm to (25.0, 3.50), turned to -90 degrees
- moved C12 17.0 mm to (26.1, 17.5), turned to 180 degrees
- moved U1 16.7 mm to (29.3, 17.2), turned to 0 degrees
- moved C14 15.0 mm to (26.1, 16.5), turned to 180 degrees
- moved L1 9.75 mm to (29.1, 13.8), turned to 180 degrees
- moved C900 8.74 mm to (29.4, 11.5), turned to 180 degrees
- moved C42 0.91 mm to (26.4, -13.9)
- moved D42 0.91 mm to (28.5, -13.5)
- moved R42 0.91 mm to (27.4, -13.9)
- moved R43 0.91 mm to (26.9, -12.5)
Routing:
- net VCC: track 68.7 -> 91.6 mm, vias 0 -> 2
- net /IE-PHASES/IE-FETS-2B/SHx: track 63.4 -> 49.2 mm
- net +3V3: track 169.4 -> 159.3 mm, vias 22 -> 21
- net /IE-PHASES/IE-FETS-2C/SHx: track 40.7 -> 50.1 mm
- net SWCLK: track 59.8 -> 50.8 mm, vias 2 -> 1
- net SWDIO: track 59.2 -> 51.2 mm, vias 2 -> 1
- net Net-(U1-LX): track 0.00 -> 2.51 mm
- net GND: track 102.9 -> 100.9 mm, vias 131 -> 130
- net Net-(U1-BS): track 6.80 -> 5.03 mm
- net ENC_2A: track 93.3 -> 92.1 mm
- net ENC_2C: track 82.2 -> 81.1 mm
- net ENC_2B: track 90.6 -> 89.5 mm
- net +5V: track 175.4 -> 176.3 mm
- net Net-(U4-PG10): track 59.6 -> 60.4 mm
- net OPAMP5_VOUT: track 65.6 -> 64.9 mm
Other:
- board text added: "INPUT"
- board text added: "OUTPUT"
- board text removed: "BATTERY"

Commit message: update for summer 2026 production run
Parts:
- J5: value Encoder1 -> Encoder
- J6: value 5V out -> Screw_Terminal_01x02
- J7: value VIN_TERMINAL -> Screw_Terminal_01x02
- J8: value Encoder2 -> Encoder
- SW1: value reset -> button; footprint AlfredoFootprints:Button_SKRKAEE020 -> AlfredoFootprints:button-3.6x6mm
- SW2: value boot-red -> button
- SW3: value user1-white -> button
- moved D42 27.7 mm to (1.04, -10.1), turned to -90 degrees
- moved R42 25.6 mm to (2.15, -9.70), turned to 90 degrees
- moved R43 24.3 mm to (2.65, -11.1), turned to 0 degrees
- moved C42 23.6 mm to (3.15, -9.70), turned to -90 degrees
- moved R67 4.50 mm to (-27.6, 16.7)
- moved SW1 2.41 mm to (27.8, -15.8)
- moved J13 1.30 mm to (29.2, -8.40)
- moved SW3 0.10 mm to (-30.0, 16.1)
Routing:
- net sVLT_VRAW: track 39.0 -> 16.6 mm
- net GND: track 100.9 -> 93.3 mm, vias 130 -> 131
- net USER1: track 50.3 -> 54.1 mm
- net Net-(U4-PG10): track 60.4 -> 58.6 mm
- net VCC: track 91.6 -> 92.5 mm, vias 2 -> 4
