File: IE-Fets.kicad_sch (KiCad schematic)
At the start: 11 parts

Commit message: schematic fix before re-org
Parts:
- renumbered Q1 to Q4, R1 to R11, R3 to R12, R4 to R13, R6 to R14, R7 to R15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

Commit message: push before schematic cleanup
Parts:
- renumbered Q4 to Q1, R11 to R1, R16 to R10, R17 to R11, R18 to R12, R12 to R3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
