File: IE-Fets.kicad_sch (KiCad schematic)
At the start: 11 parts

Commit message: updates for production run 2
Parts:
- Q4: value ~ -> (none)

Commit message: update for summer 2026 production run
Parts:
- C1: LCSC C29823 -> C380366
- D1: LCSC C131795 -> C20612286
Changed lines of the file:
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@@
 			)
 		)
-		(property "LCSC" "C131795 "
+		(property "LCSC" "C20612286"
 			(at 222.25 109.22 0)
 			(hide yes)
@@
 			)
 		)
-		(property "LCSC" "C29823"
+		(property "LCSC" "C380366"
 			(at 90.17 92.71 0)
 			(hide yes)
