File: IE-Phases.kicad_sch (KiCad schematic)
At the start: 23 parts, among them J1 JST SR/SZ, J11 Barrel_Jack, J12 JST SR/SZ, J2 Screw_Terminal_01x02, J3 Screw_Terminal_01x02, J4 Screw_Terminal_01x02, J9 JST SR/SZ, U12 FD8288T (DRV8300), U2 FD8288T (DRV8300)

Commit message: Refactor net naming and update component values
Parts:
- D15, D16, D17, D4, D5, D6: LCSC C139439 -> C558448
Changed lines of the file:
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@@
 			)
 		)
-		(property "Datasheet" "https://lcsc.com/product-detail/Schottky-Barrier-Diodes-SBD_Diodes-Incorporated-Diodes-Incorporated-SDM20U40-7_C139439.html"
+		(property "Datasheet" ""
 			(at 133.35 105.41 0)
 			(effects
@@
 			)
 		)
-		(property "LCSC" "C139439"
+		(property "LCSC" "C558448 "
 			(at 129.54 105.41 0)
 			(effects
@@
 			)
 		)
-		(property "Datasheet" "https://lcsc.com/product-detail/Schottky-Barrier-Diodes-SBD_Diodes-Incorporated-Diodes-Incorporated-SDM20U40-7_C139439.html"
+		(property "Datasheet" ""
 			(at 129.54 105.41 0)
 			(effects
@@
 			)
 		)
-		(property "LCSC" "C139439"
+		(property "LCSC" "C558448 "
 			(at 125.73 105.41 0)
 			(effects
@@
 			)
 		)
-		(property "Datasheet" "https://lcsc.com/product-detail/Schottky-Barrier-Diodes-SBD_Diodes-Incorporated-Diodes-Incorporated-SDM20U40-7_C139439.html"
+		(property "Datasheet" ""
 			(at 133.35 39.37 0)
 			(effects
@@
 			)
 		)
-		(property "LCSC" "C139439"
+		(property "LCSC" "C558448 "
 			(at 129.54 39.37 0)
 			(effects
@@
 			)
 		)
-		(property "Datasheet" "https://lcsc.com/product-detail/Schottky-Barrier-Diodes-SBD_Diodes-Incorporated-Diodes-Incorporated-SDM20U40-7_C139439.html"
+		(property "Datasheet" ""
 			(at 125.73 105.41 0)
 			(effects
@@
 			)
 		)
-		(property "LCSC" "C139439"
+		(property "LCSC" "C558448 "
 			(at 121.92 105.41 0)
 			(effects
@@
 			)
 		)
-		(property "Datasheet" "https://lcsc.com/product-detail/Schottky-Barrier-Diodes-SBD_Diodes-Incorporated-Diodes-Incorporated-SDM20U40-7_C139439.html"
+		(property "Datasheet" ""
 			(at 125.73 39.37 0)
 			(effects
@@
 			)
 		)
-		(property "LCSC" "C139439"
+		(property "LCSC" "C558448 "
 			(at 121.92 39.37 0)
 			(effects
@@
 			)
 		)
-		(property "Datasheet" "https://lcsc.com/product-detail/Schottky-Barrier-Diodes-SBD_Diodes-Incorporated-Diodes-Incorporated-SDM20U40-7_C139439.html"
+		(property "Datasheet" ""
 			(at 129.54 39.37 0)
 			(effects
@@
 			)
 		)
-		(property "LCSC" "C139439"
+		(property "LCSC" "C558448 "
 			(at 125.73 39.37 0)
 			(effects

Commit message: Add decoupling capacitor to PG10 and update footprints
Added C17 (100nF, 50V) capacitor to PG10 for improved decoupling. Updated several footprint and property fields, fixed layer and sheetname attributes, and made minor net and pad stack changes for consistency with KiCAD 9.0. Updated LCSC part number for JST SH connector.
Parts:
- removed J11: Barrel_Jack, AlfredoFootprints:DC-005C_1, symbol Connector:Barrel_Jack
- added J6: 5V out, AlfredoFootprints:TerminalBlock_Ningbo_2P_5mm, symbol Connector:Screw_Terminal_01x02
- J1, J12, J9: LCSC C160392 -> C3029336
- J2, J3, J4: LCSC C557646 -> C8404
Connections:
- net +5V: now also J6.2 (Pin_2)
- net GND: now also J6.1 (Pin_1)
