File: IE-Phases.kicad_sch (KiCad schematic)
At the start: 23 parts, among them J1 JST SR/SZ, J12 JST SR/SZ, J2 Screw_Terminal_01x02, J3 Screw_Terminal_01x02, J4 Screw_Terminal_01x02, J6 5V out, J9 JST SR/SZ, U12 FD8288T (DRV8300), U2 FD8288T (DRV8300)

Commit message: updates for production run 2
Parts:
- added J11: VIN_BARREL, AlfredoFootprints:DC-005C_1, symbol Connector:Barrel_Jack
Connections:
- net GND: now also J11.2
- net IE-FETS-2C/VOUT: now also J11.1
Other:
- moved on the sheet: J6

Commit message: update for summer 2026 production run
Parts:
- C10, C37: LCSC C13585 -> C7432781
- D15, D16, D17, D4, D5, D6: now not fitted
- J2, J3, J4: LCSC C8404 -> C557646
- J6: value 5V out -> Screw_Terminal_01x02; LCSC C8404 -> C557646
- U12, U2: LCSC C97683 -> C3036056
Changed lines of the file:
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@@
 		(on_board yes)
 		(in_pos_files yes)
-		(dnp no)
+		(dnp yes)
 		(property "Reference" "D17"
 			(at 128.27 102.87 90)
@@
 			)
 		)
-		(property "LCSC" "C8404 "
+		(property "LCSC" "C557646"
 			(at 220.98 90.17 0)
 			(hide yes)
@@
 			)
 		)
-		(property "Value" "5V out"
+		(property "Value" "Screw_Terminal_01x02"
 			(at 257.81 71.12 0)
 			(show_name no)
@@
 			)
 		)
-		(property "LCSC" "C8404 "
+		(property "LCSC" "C557646"
 			(at 255.27 73.66 0)
 			(hide yes)
@@
 		(on_board yes)
 		(in_pos_files yes)
-		(dnp no)
+		(dnp yes)
 		(property "Reference" "D16"
 			(at 124.46 102.87 90)
@@
 			)
 		)
-		(property "Datasheet" "https://static.qingshow.net/fortiortech/file/1597746029372.pdf"
+		(property "Datasheet" ""
 			(at 83.82 55.88 0)
 			(hide yes)
@@
 			)
 		)
-		(property "LCSC" "C97683"
+		(property "LCSC" "C3036056"
 			(at 101.6 72.39 0)
 			(hide yes)
@@
 		(on_board yes)
 		(in_pos_files yes)
-		(dnp no)
+		(dnp yes)
 		(property "Reference" "D6"
 			(at 128.27 36.83 90)
@@
 		(on_board yes)
 		(in_pos_files yes)
-		(dnp no)
+		(dnp yes)
 		(property "Reference" "D15"
 			(at 120.65 102.87 90)
@@
 		(on_board yes)
 		(in_pos_files yes)
-		(dnp no)
+		(dnp yes)
 		(property "Reference" "D4"
 			(at 120.65 36.83 90)
@@
 			)
 		)
-		(property "Datasheet" "https://lcsc.com/product-detail/null_C13585.html"
+		(property "Datasheet" ""
 			(at 93.98 38.1 0)
 			(hide yes)
@@
 			)
 		)
-		(property "LCSC" "C13585"
+		(property "LCSC" "C7432781"
 			(at 93.98 38.1 0)
 			(hide yes)
@@
 			)
 		)
-		(property "LCSC" "C8404 "
+		(property "LCSC" "C557646"
 			(at 220.98 96.52 0)
 			(hide yes)
@@
 			)
 		)
-		(property "Datasheet" "https://lcsc.com/product-detail/null_C13585.html"
+		(property "Datasheet" ""
 			(at 93.98 104.14 0)
 			(hide yes)
@@
 			)
 		)
-		(property "LCSC" "C13585"
+		(property "LCSC" "C7432781"
 			(at 93.98 104.14 0)
 			(hide yes)
@@
 			)
 		)
-		(property "Datasheet" "https://static.qingshow.net/fortiortech/file/1597746029372.pdf"
+		(property "Datasheet" ""
 			(at 83.82 121.92 0)
 			(hide yes)
@@
 			)
 		)
-		(property "LCSC" "C97683"
+		(property "LCSC" "C3036056"
 			(at 101.6 138.43 0)
 			(hide yes)
@@
 			)
 		)
-		(property "LCSC" "C8404 "
+		(property "LCSC" "C557646"
 			(at 220.98 102.87 0)
 			(hide yes)
@@
 		(on_board yes)
 		(in_pos_files yes)
-		(dnp no)
+		(dnp yes)
 		(property "Reference" "D5"
 			(at 124.46 36.83 90)

Commit message: fixed LCSC Numbers, order 9-10-26
Parts:
- D15, D16, D17, D4, D5, D6: LCSC C558448 -> C558448
Changed lines of the file:
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@@
 			)
 		)
-		(property "LCSC" "C558448 "
+		(property "LCSC" "C558448"
 			(at 129.54 105.41 0)
 			(hide yes)
@@
 			)
 		)
-		(property "LCSC" "C558448 "
+		(property "LCSC" "C558448"
 			(at 125.73 105.41 0)
 			(hide yes)
@@
 			)
 		)
-		(property "LCSC" "C558448 "
+		(property "LCSC" "C558448"
 			(at 129.54 39.37 0)
 			(hide yes)
@@
 			)
 		)
-		(property "LCSC" "C558448 "
+		(property "LCSC" "C558448"
 			(at 121.92 105.41 0)
 			(hide yes)
@@
 			)
 		)
-		(property "LCSC" "C558448 "
+		(property "LCSC" "C558448"
 			(at 121.92 39.37 0)
 			(hide yes)
@@
 			)
 		)
-		(property "LCSC" "C558448 "
+		(property "LCSC" "C558448"
 			(at 125.73 39.37 0)
 			(hide yes)
