File: IE-USB.kicad_sch (KiCad schematic)
At the start: 9 parts, among them U10 USBLC6-2P6, U9 USB_C_Receptacle

Commit message: Add decoupling capacitor to PG10 and update footprints
Added C17 (100nF, 50V) capacitor to PG10 for improved decoupling. Updated several footprint and property fields, fixed layer and sheetname attributes, and made minor net and pad stack changes for consistency with KiCAD 9.0. Updated LCSC part number for JST SH connector.
Parts:
- JP2: now not fitted; now left out of the parts list
Changed lines of the file:
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@@
 (kicad_sch
-	(version 20231120)
+	(version 20250114)
 	(generator "eeschema")
-	(generator_version "8.0")
+	(generator_version "9.0")
 	(paper "A4")
 	(title_block
@@
 	(label "V_USB"
 		(at 127 76.2 0)
-		(fields_autoplaced yes)
 		(effects
 			(font
@@
 		(shape input)
 		(at 186.69 60.96 0)
-		(fields_autoplaced yes)
 		(effects
 			(font
@@
 		(unit 1)
 		(exclude_from_sim yes)
-		(in_bom yes)
+		(in_bom no)
 		(on_board yes)
-		(dnp no)
+		(dnp yes)
 		(property "Reference" "JP2"
 			(at 182.118 53.34 0)
