File: I3ESC-panelized/I3ESC-panelized.kicad_pcb (KiCad board)
At the start: 4 copper layers, 208 x 222 mm, 1860 parts, among them J1 JST SR/SZ, J10 VIN_BARREL, J11 VIN_BARREL, J12 JST SR/SZ, J13 Conn_01x03, J2 Screw_Terminal_01x02, J3 Screw_Terminal_01x02, J4 Screw_Terminal_01x02, J5 Encoder, J6 Screw_Terminal_01x02, J7 Screw_Terminal_01x02, J8 Encoder, J9 JST SR/SZ, SW1 button, SW2 button, SW3 button, U1 SY8113BADC, U10 USBLC6-2P6, U11 Qwiic2, U12 FD8288T (DRV8300), U2 FD8288T (DRV8300), U3 SPX3819M5-L-3-3, U4 STM32G474RETx, U5 Qwiic1, U8 ABM3B-8.000MHZ, U9 USB_C_Receptacle

Commit message: production run 4 updates
Other:
- board size 208 x 222 mm -> 198 x 222 mm
- board text added: "1A"
- board text added: "1B"
- board text added: "1C"
- board text added: "2A"
- board text added: "2B"
- board text added: "2C"
- board text added: "BOOT"
- board text added: "MODE"
